File: pcb/STM32.sch (KiCad schematic (older format))
At the start: 11 parts

Commit message: almost finished with pcb design
Parts:
- gave numbers to parts that had none: 3
Connections:
- net labels added: 16/SCL, 17/SDA, 18/EXTRA, 19/STATUS
- net labels removed: 17/SCL, 18/SDA, 19/EXTRA, 20/STATUS, 22, 6/BUT
- wire segments 119 -> 136
Changed lines of the file:
@@
-EESchema Schematic File Version 2  date Fri 01 Feb 2013 05:54:58 PM PST
+EESchema Schematic File Version 2  date Thu 28 Feb 2013 03:25:20 PM PST
 LIBS:power
 LIBS:device
@@
 $Descr A4 11700 8267
 encoding utf-8
-Sheet 4 4
+Sheet 5 5
 Title ""
-Date "2 feb 2013"
+Date "28 feb 2013"
 Rev ""
 Comp ""
@@
 Connection ~ 9560 1545
 Wire Wire Line
-	9560 1645 9560 1195
+	9560 1645 9560 1545
+Wire Wire Line
+	9560 1545 9560 1195
 Wire Wire Line
 	8230 1700 8230 1545
@@
 	1600 6765 1600 6825
 Wire Wire Line
-	10544 4899 10130 4900
-Wire Wire Line
 	9080 4900 10130 4900
 Wire Wire Line
@@
 Wire Wire Line
 	3030 6000 3130 6000
-Connection ~ 4830 6495
 Wire Wire Line
 	3980 6495 4830 6495
@@
 	3580 6760 3580 6895
 Wire Wire Line
-	4830 6595 4830 6400
-Wire Wire Line
-	5530 1600 6530 1600
+	4830 6495 4830 6400
+Wire Wire Line
+	5530 1600 5630 1600
+Wire Wire Line
+	5630 1600 5730 1600
+Wire Wire Line
+	5730 1600 5830 1600
+Wire Wire Line
+	5830 1600 5930 1600
+Wire Wire Line
+	5930 1600 6130 1600
+Wire Wire Line
+	6130 1600 6230 1600
+Wire Wire Line
+	6230 1600 6330 1600
+Wire Wire Line
+	6330 1600 6430 1600
+Wire Wire Line
+	6430 1600 6530 1600
 Wire Wire Line
 	5530 1600 5530 1700
@@
 	6330 1600 6330 1700
 Wire Wire Line
-	6730 1600 7730 1600
+	6730 1600 6830 1600
+Wire Wire Line
+	6830 1600 6930 1600
+Wire Wire Line
+	6930 1600 7030 1600
+Wire Wire Line
+	7030 1600 7130 1600
+Wire Wire Line
+	7130 1600 7330 1600
+Wire Wire Line
+	7330 1600 7430 1600
+Wire Wire Line
+	7430 1600 7530 1600
+Wire Wire Line
+	7530 1600 7630 1600
+Wire Wire Line
+	7630 1600 7730 1600
 Connection ~ 7630 1600
 Wire Wire Line
@@
 	6030 1700 6030 1470
 Wire Wire Line
-	3580 6895 4080 6895
+	3580 6895 3980 6895
+Wire Wire Line
+	3980 6895 4080 6895
 Connection ~ 3980 6895
 Wire Wire Line
@@
 Wire Wire Line
 	10130 4900 10130 4795
-Connection ~ 10130 4900
-Wire Wire Line
-	1600 6825 2260 6825
+Wire Wire Line
+	1600 6825 1940 6825
 Wire Wire Line
 	3035 3200 3130 3200
@@
 	0    -1   -1   0
 $EndComp
-Text GLabel 10544 4899 2    60   BiDi ~ 0
-22
-$Comp
-L R R?
+$Comp
+L R R3
 U 1 1 510B216F
 P 10130 4545
-F 0 "R?" V 10210 4545 50  0000 C CNN
+F 0 "R3" V 10210 4545 50  0000 C CNN
 F 1 "1k" V 10130 4545 50  0000 C CNN
 F 4 "P1.0KJCT-ND" V 10130 4545 60  0001 C CNN "Digikey P/N"
@@
 $EndComp
 $Comp
-L LED D?
+L LED D4
 U 1 1 510B216E
 P 10330 4193
-F 0 "D?" H 10330 4293 50  0000 C CNN
+F 0 "D4" H 10330 4293 50  0000 C CNN
 F 1 "LED" H 10330 4093 50  0000 C CNN
 F 4 "P13484CT-ND" H 10330 4193 60  0001 C CNN "Digikey P/N"
@@
 $EndComp
 $Comp
-L GND #PWR?
+L GND #PWR65
 U 1 1 510B216D
 P 10630 4293
-F 0 "#PWR?" H 10630 4293 30  0001 C CNN
+F 0 "#PWR65" H 10630 4293 30  0001 C CNN
 F 1 "GND" H 10630 4223 30  0001 C CNN
 	1    10630 4293
@@
 $EndComp
 $Comp
-L STM32F103ZE U?
+L STM32F103ZE U5
 U 1 1 5109CC02
 P 6030 3750
-F 0 "U?" H 3380 5650 60  0000 C CNN
+F 0 "U5" H 3380 5650 60  0000 C CNN
 F 1 "STM32F103ZE" H 6030 3750 60  0000 C CNN
 	1    6030 3750
@@
 $EndComp
 $Comp
-L GND #PWR?
+L GND #PWR62
 U 1 1 510B1EA9
 P 7230 1500
-F 0 "#PWR?" H 7230 1500 30  0001 C CNN
+F 0 "#PWR62" H 7230 1500 30  0001 C CNN
 F 1 "GND" H 7230 1430 30  0001 C CNN
 	1    7230 1500
@@
 $EndComp
 $Comp
-L VCC #PWR?
+L VCC #PWR61
 U 1 1 510B1E7E
 P 6030 1470
-F 0 "#PWR?" H 6030 1570 30  0001 C CNN
+F 0 "#PWR61" H 6030 1570 30  0001 C CNN
 F 1 "VCC" H 6030 1570 30  0000 C CNN
 	1    6030 1470
@@
 $EndComp
 $Comp
-L VAA #PWR?
+L VAA #PWR59
 U 1 1 510B1E3B
 P 4930 1593
-F 0 "#PWR?" H 4930 1653 30  0001 C CNN
+F 0 "#PWR59" H 4930 1653 30  0001 C CNN
 F 1 "VAA" H 4930 1703 30  0000 C CNN
 	1    4930 1593
@@
 $EndComp
 $Comp
-L GND #PWR?
+L GND #PWR60
 U 1 1 510B1E3A
 P 5230 1593
-F 0 "#PWR?" H 5230 1593 30  0001 C CNN
+F 0 "#PWR60" H 5230 1593 30  0001 C CNN
 F 1 "GND" H 5230 1523 30  0001 C CNN
 	1    5230 1593
@@
 JTAG-TRST
 $Comp
-L GND #PWR?
+L GND #PWR56
 U 1 1 510B1B6F
 P 2228 4000
-F 0 "#PWR?" H 2228 4000 30  0001 C CNN
+F 0 "#PWR56" H 2228 4000 30  0001 C CNN
 F 1 "GND" H 2228 3930 30  0001 C CNN
 	1    2228 4000
@@
 R9
 Text GLabel 3031 3700 0    60   BiDi ~ 0
-19/EXTRA
+18/EXTRA
 Text GLabel 3031 3800 0    60   BiDi ~ 0
-20/STATUS
+19/STATUS
 Text GLabel 3029 4400 0    60   BiDi ~ 0
-18/SDA
+17/SDA
 Text GLabel 3029 4300 0    60   BiDi ~ 0
-17/SCL
+16/SCL
 Text GLabel 9177 2700 2    60   BiDi ~ 0
 15/MC15
@@
 Text GLabel 3030 5600 0    60   BiDi ~ 0
 2/MC2
-Text GLabel 4830 6595 3    60   BiDi ~ 0
-6/BUT
 Text Notes 3100 1410 0    40   ~ 0
 solder jumper
@@
 P 2948 1100
 AR Path="/51099A3F/4D52E865" Ref="#PWR054"  Part="1"
-AR Path="/510998BD/4D52E865" Ref="#PWR054"  Part="1"
-F 0 "#PWR054" H 2948 1160 30  0001 C CNN
+AR Path="/510998BD/4D52E865" Ref="#PWR57"  Part="1"
+F 0 "#PWR57" H 2948 1160 30  0001 C CNN
 F 1 "VAA" H 2948 1210 30  0000 C CNN
 	1    2948 1100
@@
 Text GLabel 7930 1593 1    60   BiDi ~ 0
 RST
-Text GLabel 2260 6825 2    60   BiDi ~ 0
+Text GLabel 1940 6825 2    60   BiDi ~ 0
 RST
 Text Label 8030 943  3    60   ~ 0
@@
 P 3580 6760
 AR Path="/51099A3F/4B8ADEC7" Ref="#PWR061"  Part="1"
-AR Path="/510998BD/4B8ADEC7" Ref="#PWR061"  Part="1"
-F 0 "#PWR061" H 3580 6860 30  0001 C CNN
+AR Path="/510998BD/4B8ADEC7" Ref="#PWR58"  Part="1"
+F 0 "#PWR58" H 3580 6860 30  0001 C CNN
 F 1 "VCC" H 3580 6860 30  0000 C CNN
 	1    3580 6760
@@
 P 9560 1645
 AR Path="/51099A3F/4B8383A4" Ref="#PWR062"  Part="1"
-AR Path="/510998BD/4B8383A4" Ref="#PWR062"  Part="1"
-F 0 "#PWR062" H 9560 1645 30  0001 C CNN
+AR Path="/510998BD/4B8383A4" Ref="#PWR64"  Part="1"
+F 0 "#PWR64" H 9560 1645 30  0001 C CNN
 F 1 "GND" H 9560 1575 30  0001 C CNN
 	1    9560 1645
@@
 P 8530 943
 AR Path="/51099A3F/4B83757E" Ref="#PWR063"  Part="1"
-AR Path="/510998BD/4B83757E" Ref="#PWR063"  Part="1"
-F 0 "#PWR063" H 8530 943 30  0001 C CNN
+AR Path="/510998BD/4B83757E" Ref="#PWR63"  Part="1"
+F 0 "#PWR63" H 8530 943 30  0001 C CNN
 F 1 "GND" H 8530 873 30  0001 C CNN
 	1    8530 943
@@
 P 1601 7325
 AR Path="/51099A3F/4B83757C" Ref="#PWR064"  Part="1"
-AR Path="/510998BD/4B83757C" Ref="#PWR064"  Part="1"
-F 0 "#PWR064" H 1601 7325 30  0001 C CNN
+AR Path="/510998BD/4B83757C" Ref="#PWR55"  Part="1"
+F 0 "#PWR55" H 1601 7325 30  0001 C CNN
 F 1 "GND" H 1601 7255 30  0001 C CNN
 	1    1601 7325
@@
 P 1600 6215
 AR Path="/51099A3F/4B83757A" Ref="#PWR065"  Part="1"
-AR Path="/510998BD/4B83757A" Ref="#PWR065"  Part="1"
-F 0 "#PWR065" H 1600 6315 30  0001 C CNN
+AR Path="/510998BD/4B83757A" Ref="#PWR54"  Part="1"
+F 0 "#PWR54" H 1600 6315 30  0001 C CNN
 F 1 "VCC" H 1600 6315 30  0000 C CNN
 	1    1600 6215

Commit message: working on power circuitry
Connections:
- wire segments 136 -> 118
Other:
- note removed: "solder jumper"
Changed lines of the file:
@@
-EESchema Schematic File Version 2  date Thu 28 Feb 2013 03:25:20 PM PST
+EESchema Schematic File Version 2  date Tue 12 Mar 2013 12:56:47 AM PDT
 LIBS:power
 LIBS:device
@@
 LIBS:uln2804a
 LIBS:leaf
+LIBS:led_16x16
 LIBS:panels_g4-cache
 EELAYER 25  0
@@
 Sheet 5 5
 Title ""
-Date "28 feb 2013"
+Date "12 mar 2013"
 Rev ""
 Comp ""
@@
 Connection ~ 9560 1545
 Wire Wire Line
-	9560 1645 9560 1545
-Wire Wire Line
-	9560 1545 9560 1195
+	9560 1645 9560 1195
 Wire Wire Line
 	8230 1700 8230 1545
@@
 	4830 6495 4830 6400
 Wire Wire Line
-	5530 1600 5630 1600
-Wire Wire Line
-	5630 1600 5730 1600
-Wire Wire Line
-	5730 1600 5830 1600
-Wire Wire Line
-	5830 1600 5930 1600
-Wire Wire Line
-	5930 1600 6130 1600
-Wire Wire Line
-	6130 1600 6230 1600
-Wire Wire Line
-	6230 1600 6330 1600
-Wire Wire Line
-	6330 1600 6430 1600
-Wire Wire Line
-	6430 1600 6530 1600
+	5530 1600 6530 1600
 Wire Wire Line
 	5530 1600 5530 1700
@@
 	6330 1600 6330 1700
 Wire Wire Line
-	6730 1600 6830 1600
-Wire Wire Line
-	6830 1600 6930 1600
-Wire Wire Line
-	6930 1600 7030 1600
-Wire Wire Line
-	7030 1600 7130 1600
-Wire Wire Line
-	7130 1600 7330 1600
-Wire Wire Line
-	7330 1600 7430 1600
-Wire Wire Line
-	7430 1600 7530 1600
-Wire Wire Line
-	7530 1600 7630 1600
-Wire Wire Line
-	7630 1600 7730 1600
+	6730 1600 7730 1600
 Connection ~ 7630 1600
 Wire Wire Line
@@
 	6030 1700 6030 1470
 Wire Wire Line
-	3580 6895 3980 6895
-Wire Wire Line
-	3980 6895 4080 6895
+	3580 6895 4080 6895
 Connection ~ 3980 6895
 Wire Wire Line
@@
 $EndComp
 $Comp
-L GND #PWR65
+L GND #PWR028
 U 1 1 510B216D
 P 10630 4293
-F 0 "#PWR65" H 10630 4293 30  0001 C CNN
+F 0 "#PWR028" H 10630 4293 30  0001 C CNN
 F 1 "GND" H 10630 4223 30  0001 C CNN
 	1    10630 4293
@@
 $EndComp
 $Comp
-L GND #PWR62
+L GND #PWR029
 U 1 1 510B1EA9
 P 7230 1500
-F 0 "#PWR62" H 7230 1500 30  0001 C CNN
+F 0 "#PWR029" H 7230 1500 30  0001 C CNN
 F 1 "GND" H 7230 1430 30  0001 C CNN
 	1    7230 1500
@@
 $EndComp
 $Comp
-L VCC #PWR61
+L VCC #PWR030
 U 1 1 510B1E7E
 P 6030 1470
-F 0 "#PWR61" H 6030 1570 30  0001 C CNN
+F 0 "#PWR030" H 6030 1570 30  0001 C CNN
 F 1 "VCC" H 6030 1570 30  0000 C CNN
 	1    6030 1470
@@
 $EndComp
 $Comp
-L VAA #PWR59
+L VAA #PWR34
 U 1 1 510B1E3B
 P 4930 1593
-F 0 "#PWR59" H 4930 1653 30  0001 C CNN
+F 0 "#PWR34" H 4930 1653 30  0001 C CNN
 F 1 "VAA" H 4930 1703 30  0000 C CNN
 	1    4930 1593
@@
 $EndComp
 $Comp
-L GND #PWR60
+L GND #PWR031
 U 1 1 510B1E3A
 P 5230 1593
-F 0 "#PWR60" H 5230 1593 30  0001 C CNN
+F 0 "#PWR031" H 5230 1593 30  0001 C CNN
 F 1 "GND" H 5230 1523 30  0001 C CNN
 	1    5230 1593
@@
 JTAG-TRST
 $Comp
-L GND #PWR56
+L GND #PWR032
 U 1 1 510B1B6F
 P 2228 4000
-F 0 "#PWR56" H 2228 4000 30  0001 C CNN
+F 0 "#PWR032" H 2228 4000 30  0001 C CNN
 F 1 "GND" H 2228 3930 30  0001 C CNN
 	1    2228 4000
@@
 Text GLabel 3030 5600 0    60   BiDi ~ 0
 2/MC2
-Text Notes 3100 1410 0    40   ~ 0
-solder jumper
 $Comp
 L JP_SW JP1
@@
 P 2948 1100
 AR Path="/51099A3F/4D52E865" Ref="#PWR054"  Part="1"
-AR Path="/510998BD/4D52E865" Ref="#PWR57"  Part="1"
-F 0 "#PWR57" H 2948 1160 30  0001 C CNN
+AR Path="/510998BD/4D52E865" Ref="#PWR32"  Part="1"
+F 0 "#PWR32" H 2948 1160 30  0001 C CNN
 F 1 "VAA" H 2948 1210 30  0000 C CNN
 	1    2948 1100
@@
 P 3580 6760
 AR Path="/51099A3F/4B8ADEC7" Ref="#PWR061"  Part="1"
-AR Path="/510998BD/4B8ADEC7" Ref="#PWR58"  Part="1"
-F 0 "#PWR58" H 3580 6860 30  0001 C CNN
+AR Path="/510998BD/4B8ADEC7" Ref="#PWR033"  Part="1"
+F 0 "#PWR033" H 3580 6860 30  0001 C CNN
 F 1 "VCC" H 3580 6860 30  0000 C CNN
 	1    3580 6760
@@
 P 9560 1645
 AR Path="/51099A3F/4B8383A4" Ref="#PWR062"  Part="1"
-AR Path="/510998BD/4B8383A4" Ref="#PWR64"  Part="1"
-F 0 "#PWR64" H 9560 1645 30  0001 C CNN
+AR Path="/510998BD/4B8383A4" Ref="#PWR034"  Part="1"
+F 0 "#PWR034" H 9560 1645 30  0001 C CNN
 F 1 "GND" H 9560 1575 30  0001 C CNN
 	1    9560 1645
@@
 P 8530 943
 AR Path="/51099A3F/4B83757E" Ref="#PWR063"  Part="1"
-AR Path="/510998BD/4B83757E" Ref="#PWR63"  Part="1"
-F 0 "#PWR63" H 8530 943 30  0001 C CNN
+AR Path="/510998BD/4B83757E" Ref="#PWR035"  Part="1"
+F 0 "#PWR035" H 8530 943 30  0001 C CNN
 F 1 "GND" H 8530 873 30  0001 C CNN
 	1    8530 943
@@
 P 1601 7325
 AR Path="/51099A3F/4B83757C" Ref="#PWR064"  Part="1"
-AR Path="/510998BD/4B83757C" Ref="#PWR55"  Part="1"
-F 0 "#PWR55" H 1601 7325 30  0001 C CNN
+AR Path="/510998BD/4B83757C" Ref="#PWR036"  Part="1"
+F 0 "#PWR036" H 1601 7325 30  0001 C CNN
 F 1 "GND" H 1601 7255 30  0001 C CNN
 	1    1601 7325
@@
 P 1600 6215
 AR Path="/51099A3F/4B83757A" Ref="#PWR065"  Part="1"
-AR Path="/510998BD/4B83757A" Ref="#PWR54"  Part="1"
-F 0 "#PWR54" H 1600 6315 30  0001 C CNN
+AR Path="/510998BD/4B83757A" Ref="#PWR037"  Part="1"
+F 0 "#PWR037" H 1600 6315 30  0001 C CNN
 F 1 "VCC" H 1600 6315 30  0000 C CNN
 	1    1600 6215

Commit message: Work on single PCB version.
Parts:
- removed JP1: JP_SW, JP_SW, symbol JP_SW
Connections:
- net labels removed: VAA, VBAT, VREF
- wire segments 118 -> 131
- no-connect marks 0 -> 50
Changed lines of the file:
@@
-EESchema Schematic File Version 2  date Tue 12 Mar 2013 12:56:47 AM PDT
+EESchema Schematic File Version 2  date Tue 12 Mar 2013 12:36:21 PM PDT
 LIBS:power
 LIBS:device
@@
 LIBS:leaf
 LIBS:led_16x16
+LIBS:uA7800
 LIBS:panels_g4-cache
 EELAYER 25  0
@@
 Comment4 ""
 $EndDescr
+NoConn ~ 9080 5300
+NoConn ~ 9080 5100
+NoConn ~ 9080 5200
+NoConn ~ 9080 5400
+NoConn ~ 9080 5500
+NoConn ~ 9080 5600
+NoConn ~ 9080 5700
+NoConn ~ 9080 5800
+NoConn ~ 9080 5900
+NoConn ~ 9080 6000
+NoConn ~ 9080 6100
+NoConn ~ 9080 5000
+NoConn ~ 9080 4600
+NoConn ~ 9080 4700
+NoConn ~ 6330 6400
+NoConn ~ 6230 6400
+NoConn ~ 6130 6400
+NoConn ~ 6030 6400
+NoConn ~ 5930 6400
+NoConn ~ 5830 6400
+NoConn ~ 5730 6400
+NoConn ~ 5630 6400
+NoConn ~ 5530 6400
+NoConn ~ 5430 6400
+NoConn ~ 5330 6400
+NoConn ~ 5230 6400
+NoConn ~ 5130 6400
+NoConn ~ 5030 6400
+NoConn ~ 4930 6400
+Wire Wire Line
+	5030 1700 5030 1610
+$Comp
+L VCC #PWR?
+U 1 1 513F826F
+P 5030 1610
+F 0 "#PWR?" H 5030 1710 30  0001 C CNN
+F 1 "VCC" H 5030 1710 30  0000 C CNN
+	1    5030 1610
+	1    0    0    -1
+$EndComp
+$Comp
+L VCC #PWR?
+U 1 1 513F825E
+P 4930 1610
+F 0 "#PWR?" H 4930 1710 30  0001 C CNN
+F 1 "VCC" H 4930 1710 30  0000 C CNN
+	1    4930 1610
+	1    0    0    -1
+$EndComp
+Wire Wire Line
+	4930 1700 4930 1610
+NoConn ~ 3130 5200
+NoConn ~ 3130 5100
+NoConn ~ 3130 5000
+NoConn ~ 3130 4900
+NoConn ~ 3130 4800
+NoConn ~ 3130 4700
+NoConn ~ 3130 4600
+NoConn ~ 3130 4500
+NoConn ~ 3130 2700
+NoConn ~ 3130 2800
+NoConn ~ 3130 2900
+NoConn ~ 3130 3000
+NoConn ~ 3130 2600
+NoConn ~ 3130 2500
+NoConn ~ 3130 2400
+NoConn ~ 3130 2300
+NoConn ~ 3130 2200
+NoConn ~ 3130 2100
+NoConn ~ 3130 2000
+NoConn ~ 5130 1700
+NoConn ~ 5330 1700
 Wire Wire Line
 	8130 1700 8130 1195
 Connection ~ 9560 1545
 Wire Wire Line
-	9560 1645 9560 1195
+	9560 1645 9560 1545
+Wire Wire Line
+	9560 1545 9560 1195
 Wire Wire Line
 	8230 1700 8230 1545
@@
 	4830 6495 4830 6400
 Wire Wire Line
-	5530 1600 6530 1600
+	5530 1600 5630 1600
+Wire Wire Line
+	5630 1600 5730 1600
+Wire Wire Line
+	5730 1600 5830 1600
+Wire Wire Line
+	5830 1600 5930 1600
+Wire Wire Line
+	5930 1600 6130 1600
+Wire Wire Line
+	6130 1600 6230 1600
+Wire Wire Line
+	6230 1600 6330 1600
+Wire Wire Line
+	6330 1600 6430 1600
+Wire Wire Line
+	6430 1600 6530 1600
 Wire Wire Line
 	5530 1600 5530 1700
@@
 	6330 1600 6330 1700
 Wire Wire Line
-	6730 1600 7730 1600
+	6730 1600 6830 1600
+Wire Wire Line
+	6830 1600 6930 1600
+Wire Wire Line
+	6930 1600 7030 1600
+Wire Wire Line
+	7030 1600 7130 1600
+Wire Wire Line
+	7130 1600 7330 1600
+Wire Wire Line
+	7330 1600 7430 1600
+Wire Wire Line
+	7430 1600 7530 1600
+Wire Wire Line
+	7530 1600 7630 1600
+Wire Wire Line
+	7630 1600 7730 1600
 Connection ~ 7630 1600
 Wire Wire Line
@@
 Wire Wire Line
 	6730 1600 6730 1700
-Wire Wire Line
-	2948 1100 2948 1200
-Wire Wire Line
-	3448 1200 3648 1200
 Connection ~ 8645 1543
 Connection ~ 8645 1193
@@
 	7930 1700 7930 1593
 Wire Wire Line
-	2948 1200 3148 1200
-Wire Wire Line
-	3648 1200 3648 1100
-Wire Wire Line
 	9177 2500 9080 2500
 Wire Wire Line
@@
 	7930 6493 7930 6400
 Wire Wire Line
-	2228 4000 2228 3900
+	2358 4000 2358 3900
 Wire Wire Line
 	3028 4000 3130 4000
@@
 	3028 4100 3130 4100
 Wire Wire Line
-	2228 3900 3130 3900
+	2358 3900 3130 3900
 Wire Wire Line
 	9080 4800 9181 4800
@@
 Wire Wire Line
 	5230 1593 5230 1700
-Wire Wire Line
-	5030 1593 5030 1700
-Wire Wire Line
-	5330 1593 5330 1700
-Wire Wire Line
-	4930 1593 4930 1700
 Wire Wire Line
 	10130 4295 10130 4193
@@
 	6030 1700 6030 1470
 Wire Wire Line
-	3580 6895 4080 6895
+	3580 6895 3980 6895
+Wire Wire Line
+	3980 6895 4080 6895
 Connection ~ 3980 6895
 Wire Wire Line
@@
 $EndComp
 $Comp
-L VAA #PWR34
-U 1 1 510B1E3B
-P 4930 1593
-F 0 "#PWR34" H 4930 1653 30  0001 C CNN
-F 1 "VAA" H 4930 1703 30  0000 C CNN
-	1    4930 1593
-	1    0    0    -1
-$EndComp
-$Comp
 L GND #PWR031
 U 1 1 510B1E3A
@@
 	1    0    0    1
 $EndComp
-Text GLabel 5030 1593 1    60   BiDi ~ 0
-VREF
-Text GLabel 5330 1593 1    60   BiDi ~ 0
-VBAT
 Text GLabel 6530 6493 3    60   BiDi ~ 0
 R15
@@
 L GND #PWR032
 U 1 1 510B1B6F
-P 2228 4000
-F 0 "#PWR032" H 2228 4000 30  0001 C CNN
-F 1 "GND" H 2228 3930 30  0001 C CNN
-	1    2228 4000
+P 2358 4000
+F 0 "#PWR032" H 2358 4000 30  0001 C CNN
+F 1 "GND" H 2358 3930 30  0001 C CNN
+	1    2358 4000
 	1    0    0    -1
 $EndComp
@@
 Text GLabel 3030 5600 0    60   BiDi ~ 0
 2/MC2
-$Comp
-L JP_SW JP1
-U 1 1 4D54699B
-P 3298 1200
-AR Path="/51099A3F/4D54699B" Ref="JP1"  Part="1"
-AR Path="/510998BD/4D54699B" Ref="JP1"  Part="1"
-F 0 "JP1" H 3398 1300 50  0000 C CNN
-F 1 "JP_SW" H 3298 1100 50  0000 C CNN
-F 2 "JP_SW" H 3298 1350 50  0001 C CNN
-	1    3298 1200
-	1    0    0    -1
-$EndComp
-Text GLabel 3648 1100 1    60   BiDi ~ 0
-VREF
-$Comp
-L VAA #PWR054
-U 1 1 4D52E865
-P 2948 1100
-AR Path="/51099A3F/4D52E865" Ref="#PWR054"  Part="1"
-AR Path="/510998BD/4D52E865" Ref="#PWR32"  Part="1"
-F 0 "#PWR32" H 2948 1160 30  0001 C CNN
-F 1 "VAA" H 2948 1210 30  0000 C CNN
-	1    2948 1100
-	1    0    0    -1
-$EndComp
 Text GLabel 7930 1593 1    60   BiDi ~ 0
 RST
