File: pcb/panels_g4.sch (KiCad schematic (older format))
At the start: 46 parts, among them IC1 ATMEGA168-A, P1 CONN_8, P2 CONN_8, U1 ULN2804A

Commit message: work in progress for the pcb schematic design.
Parts:
- removed C1, C2: 0.1uF, symbol C
- removed IC1: ATMEGA168-A, TQFP32, symbol ATMEGA168-A
- removed MATRIX1, MATRIX? (x3): LED_8X8, symbol LED_8X8
- removed P1, P2: CONN_8, symbol CONN_8
- removed R1, R2, R3, R4, R5, R6, R7, R8, R? (x24): 82, symbol R
- removed U1, U? (x3): ULN2804A, symbol ULN2804A
- removed U?: STM32F407ZE, symbol STM32F407ZE
Connections:
- net labels removed: GND, VCC
- wire segments 196 -> 0
- no-connect marks 5 -> 0
Other:
- note removed: "BOTTOM"
- note removed: "TOP"

Commit message: almost finished with pcb design
Changed lines of the file:
@@
-EESchema Schematic File Version 2  date Fri 01 Feb 2013 05:54:58 PM PST
+EESchema Schematic File Version 2  date Thu 28 Feb 2013 03:25:20 PM PST
 LIBS:power
 LIBS:device
@@
 $Descr A4 11700 8267
 encoding utf-8
-Sheet 1 4
+Sheet 1 5
 Title ""
-Date "2 feb 2013"
+Date "28 feb 2013"
 Rev ""
 Comp ""
@@
 $EndDescr
 $Sheet
-S 7650 3150 2000 1400
+S 3700 3900 2000 1400
+U 511014E4
+F0 "pwr" 60
+F1 "pwr.sch" 60
+$EndSheet
+$Sheet
+S 6400 3900 2000 1400
 U 51099D6B
 F0 "LEDs" 60
@@
 $EndSheet
 $Sheet
-S 2150 3150 2000 1400
+S 3700 1900 2000 1400
 U 51099A3F
 F0 "conn" 60
@@
 $EndSheet
 $Sheet
-S 4850 3150 2000 1400
+S 6400 1900 2000 1400
 U 510998BD
 F0 "STM32" 60
