File: max6960/four_panel/20mm_matrix/driver/driver.sch (KiCad schematic (older format))
At the start: 10 parts, among them P1 LED-MATRIX-2X-8X8, P2 LED-MATRIX-2X-8X8, P3 CONN15, P4 CONN15, U1 MAX6960, U2 74AHC1G126, U3 MAX6960

Commit message: Re-routed four matrix panel driver and adapter. Switched to board-to-board connectors from major league.
Parts:
- removed P1, P2: LED-MATRIX-2X-8X8, symbol LED-MATRIX-2X-8X8
- added P1, P2: CONN15X2, symbol CONN15X2
Connections:
- net COL_A1: now also P1.18
- net COL_A10: now also P1.13
- net COL_A11: now also P1.11
- net COL_A12: now also P1.9
- net COL_A13: now also P1.7
- net COL_A14: now also P1.5
- net COL_A15: now also P1.3
- net COL_A16: now also P1.1
- net COL_A2: now also P1.20
- net COL_A3: now also P1.22
- net COL_A4: now also P1.25
- net COL_A5: now also P1.23
- net COL_A6: now also P1.21
- net COL_A7: now also P1.19
- net COL_A8: now also P1.17
- net COL_A9: now also P1.15
- net COL_B1: now also P2.18
- net COL_B10: now also P2.13
- net COL_B11: now also P2.11
- net COL_B12: now also P2.9
- net COL_B13: now also P2.7
- net COL_B14: now also P2.5
- net COL_B15: now also P2.3
- net COL_B16: now also P2.1
- net COL_B2: now also P2.20
- net COL_B3: now also P2.22
- net COL_B4: now also P2.25
- net COL_B5: now also P2.23
- net COL_B6: now also P2.21
- net COL_B7: now also P2.19
- net COL_B8: now also P2.17
- net COL_B9: now also P2.15
- net GND: now also P1.28, P1.30, P2.28, P2.30
- net ROW_A1: now also P1.2
- net ROW_A2: now also P1.4
- net ROW_A3: now also P1.6
- net ROW_A4: now also P1.8
- net ROW_A5: now also P1.10
- net ROW_A6: now also P1.12
- net ROW_A7: now also P1.14
- net ROW_A8: now also P1.16
- net ROW_B1: now also P2.2
- net ROW_B2: now also P2.4
- net ROW_B3: now also P2.6
- net ROW_B4: now also P2.8
- net ROW_B5: now also P2.10
- net ROW_B6: now also P2.12
- net ROW_B7: now also P2.14
- net ROW_B8: now also P2.16
- net VAUX: now also P1.27, P1.29, P2.27, P2.29
- net v+: now also C1.1, C2.1
- no-connect marks 2 -> 8
Other:
- note removed: "SMH102-LPSE-D18-SP-BK"
- moved on the sheet: C1, C2, C3, P3, P4, U2, U3
