File: max6960/four_panel/20mm_matrix/adapter_2_layer/adapter.kicad_pcb (KiCad board)
At the start: 2 copper layers, 40 x 40 mm, 6 parts, among them M1 BETLUX-LED-8X8_C, M2 BETLUX-LED-8X8_C, M3 BETLUX-LED-8X8_C, M4 BETLUX-LED-8X8_C, P1 CONN15X2, P2 CONN15X2

Commit message: Created gerber files and BOM for 4-matrix atmega328 and max6960 PCBs.
Other:
- board text added: "4-Matrix Max6960 Adapter v0.1 www.iorodeo.com"
- board text added: "K1"
- board text added: "K2"
- board text added: "K3"
- board text added: "K4"
- board text added: "K5"
- board text added: "K6"
- board text added: "K7"
- board text added: "K8"
Changed lines of the file:
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@@
     (area 49.721799 49.721799 90.278201 90.278201)
     (thickness 1.6)
-    (drawings 6)
+    (drawings 15)
     (tracks 413)
     (zones 0)
@@
     (visible_elements FFFFFF7F)
     (pcbplotparams
-      (layerselection 3178497)
+      (layerselection 284196865)
       (usegerberextensions true)
       (excludeedgelayer true)
@@
       (outputformat 1)
       (mirror false)
-      (drillshape 1)
+      (drillshape 0)
       (scaleselection 1)
-      (outputdirectory ""))
+      (outputdirectory gerber_v0p1/))
   )
   (net 0 "")
@@
     )
   )
+  (gr_text K8 (at 89.2429 88.8873 90) (layer F.SilkS)
+    (effects (font (size 1.016 1.016) (thickness 0.2032)))
+  )
+  (gr_text K7 (at 70.8025 88.9254 90) (layer F.SilkS)
+    (effects (font (size 1.016 1.016) (thickness 0.2032)))
+  )
+  (gr_text K6 (at 89.2556 51.0794 90) (layer F.SilkS)
+    (effects (font (size 1.016 1.016) (thickness 0.2032)))
+  )
+  (gr_text K5 (at 70.8533 51.0667 90) (layer F.SilkS)
+    (effects (font (size 1.016 1.016) (thickness 0.2032)))
+  )
+  (gr_text K4 (at 69.2531 88.9254 90) (layer F.SilkS)
+    (effects (font (size 1.016 1.016) (thickness 0.2032)))
+  )
+  (gr_text K3 (at 50.8508 88.8873 90) (layer F.SilkS)
+    (effects (font (size 1.016 1.016) (thickness 0.2032)))
+  )
+  (gr_text K2 (at 69.2658 51.0794 90) (layer F.SilkS)
+    (effects (font (size 1.016 1.016) (thickness 0.2032)))
+  )
+  (gr_text K1 (at 50.8381 51.308 90) (layer F.SilkS)
+    (effects (font (size 1.016 1.016) (thickness 0.2032)))
+  )
+  (gr_text "4-Matrix \nMax6960 \nAdapter v0.1\nwww.iorodeo.com" (at 59.9694 51.2826) (layer B.SilkS)
+    (effects (font (size 1.016 1.016) (thickness 0.2032)) (justify mirror))
+  )
   (gr_text BOT (at 84 88.5) (layer B.SilkS)
