File: atmega328/four_panel/20mm_matrix/ver3/test_arena/arena.kicad_pcb (KiCad board)
At the start: 2 copper layers, 260 x 60 mm, 39 parts, among them M1 VAL**, M2 VAL**, M3 VAL**, M4 VAL**, M5 VAL**, M6 VAL**, P1 CONN15, P10 CONN_20X2, P2 CONN15, P3 CONN15, P4 CONN15, P5 CONN15, P6 CONN15, P7 CONN_20X2, P8 CONN_34X2, P9 CONN_2, Q1 MOSFET_NCHAN, SW1 SWITCH_INV, U1 SPARKFUN_TXB0104, U2 SPARKFUN_TXB0104, U3 SPARKFUN_TXB0104, U4 SPARKFUN_TXB0104, U5 SPARKFUN_TXB0104, U6 SPARKFUN_TXB0104, U7 SPARKFUN_TXB0104, U8 POLOLU_3V3

Commit message: Modified routing.
Routing:
- net /SCK_0_3V3: track 220.4 -> 218.4 mm
- net /CS_6_5V: track 243.1 -> 242.0 mm
- net /MOSI_2_3V3: track 174.8 -> 174.3 mm

Commit message: Added gerber files for v0.3 of the g4 test arena.
Other:
- board text added: "4x 20mm Atmega328 Test Arena v0.3 R1 www.iorodeo.com"
- board text removed: "4x 20mm Atmega328 Test Arena v0.3 www.iorodeo.com"
Changed lines of the file:
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@@
     (links 232)
     (no_connects 0)
-    (area 39.749999 49.527499 311.182656 113.7284)
+    (area 39.749999 49.527499 315.466998 121.699006)
     (thickness 1.6)
-    (drawings 9)
+    (drawings 11)
     (tracks 1360)
     (zones 0)
@@
       (drillshape 0)
       (scaleselection 1)
-      (outputdirectory gerber_v0p2_rev1/))
+      (outputdirectory gerber_r1/))
   )
   (net 0 "")
@@
   (net 71 /SCK_5_5V)
   (net 72 GND)
-  (net 73 N-00000100)
-  (net 74 N-00000103)
-  (net 75 N-0000028)
-  (net 76 N-0000029)
-  (net 77 N-0000030)
-  (net 78 N-0000032)
-  (net 79 N-0000077)
+  (net 73 N-00000108)
+  (net 74 N-0000029)
+  (net 75 N-0000034)
+  (net 76 N-0000086)
+  (net 77 N-0000089)
+  (net 78 N-0000093)
+  (net 79 N-0000098)
   (net_class Default "This is the default net class."
     (clearance 0.254)
@@
     (add_net /SCK_5_3V3)
     (add_net /SCK_5_5V)
-    (add_net N-00000100)
-    (add_net N-00000103)
-    (add_net N-0000028)
+    (add_net N-00000108)
     (add_net N-0000029)
-    (add_net N-0000030)
-    (add_net N-0000032)
-    (add_net N-0000077)
+    (add_net N-0000034)
+    (add_net N-0000086)
+    (add_net N-0000089)
+    (add_net N-0000093)
+    (add_net N-0000098)
   )
   (net_class Pwr ""
@@
     (pad 1 smd rect (at -0.9525 1.09982 90) (size 0.8001 1.00076)
       (layers F.Cu F.Paste F.Mask)
-      (net 75 N-0000028)
+      (net 74 N-0000029)
     )
     (model smd\SOT23_3.wrl
@@
     (pad 2 smd rect (at 0.9525 0 180) (size 0.889 1.397)
       (layers F.Cu F.Paste F.Mask)
-      (net 75 N-0000028)
+      (net 74 N-0000029)
     )
     (model smd/chip_cms.wrl
@@
     (pad 1 smd rect (at -0.9525 0 90) (size 0.889 1.397)
       (layers F.Cu F.Paste F.Mask)
-      (net 75 N-0000028)
+      (net 74 N-0000029)
     )
     (pad 2 smd rect (at 0.9525 0 90) (size 0.889 1.397)
@@
     (pad 4 thru_hole circle (at -5.08 0 90) (size 1.778 1.778) (drill 1.016)
       (layers *.Cu *.Mask F.SilkS)
-      (net 74 N-00000103)
+      (net 75 N-0000034)
     )
     (pad 5 thru_hole circle (at -5.08 2.54 90) (size 1.778 1.778) (drill 1.016)
@@
     (pad 4 thru_hole circle (at -5.08 0 90) (size 1.778 1.778) (drill 1.016)
       (layers *.Cu *.Mask F.SilkS)
-      (net 77 N-0000030)
+      (net 79 N-0000098)
     )
     (pad 5 thru_hole circle (at -5.08 2.54 90) (size 1.778 1.778) (drill 1.016)
@@
     (pad 4 thru_hole circle (at -5.08 0 90) (size 1.778 1.778) (drill 1.016)
       (layers *.Cu *.Mask F.SilkS)
-      (net 78 N-0000032)
+      (net 73 N-00000108)
     )
     (pad 5 thru_hole circle (at -5.08 2.54 90) (size 1.778 1.778) (drill 1.016)
@@
     (pad 4 thru_hole circle (at -5.08 0 90) (size 1.778 1.778) (drill 1.016)
       (layers *.Cu *.Mask F.SilkS)
-      (net 79 N-0000077)
+      (net 77 N-0000089)
     )
     (pad 5 thru_hole circle (at -5.08 2.54 90) (size 1.778 1.778) (drill 1.016)
@@
     (pad 4 thru_hole circle (at -5.08 0 90) (size 1.778 1.778) (drill 1.016)
       (layers *.Cu *.Mask F.SilkS)
-      (net 76 N-0000029)
+      (net 78 N-0000093)
     )
     (pad 5 thru_hole circle (at -5.08 2.54 90) (size 1.778 1.778) (drill 1.016)
@@
     (pad 4 thru_hole circle (at -5.08 0 90) (size 1.778 1.778) (drill 1.016)
       (layers *.Cu *.Mask F.SilkS)
-      (net 73 N-00000100)
+      (net 76 N-0000086)
     )
     (pad 5 thru_hole circle (at -5.08 2.54 90) (size 1.778 1.778) (drill 1.016)
@@
     (pad 1 thru_hole circle (at -2.5 0 270) (size 1.5 1.5) (drill 1)
       (layers *.Cu *.Mask F.SilkS)
-      (net 74 N-00000103)
+      (net 75 N-0000034)
     )
     (pad 2 thru_hole circle (at 2.5 0 270) (size 1.5 1.5) (drill 1)
@@
     (pad 1 thru_hole circle (at -2.5 0 270) (size 1.5 1.5) (drill 1)
       (layers *.Cu *.Mask F.SilkS)
-      (net 77 N-0000030)
+      (net 79 N-0000098)
     )
     (pad 2 thru_hole circle (at 2.5 0 270) (size 1.5 1.5) (drill 1)
@@
     (pad 1 thru_hole circle (at -2.5 0 270) (size 1.5 1.5) (drill 1)
       (layers *.Cu *.Mask F.SilkS)
-      (net 78 N-0000032)
+      (net 73 N-00000108)
     )
     (pad 2 thru_hole circle (at 2.5 0 270) (size 1.5 1.5) (drill 1)
@@
     (pad 1 thru_hole circle (at -2.5 0 270) (size 1.5 1.5) (drill 1)
       (layers *.Cu *.Mask F.SilkS)
-      (net 79 N-0000077)
+      (net 77 N-0000089)
     )
     (pad 2 thru_hole circle (at 2.5 0 270) (size 1.5 1.5) (drill 1)
@@
     (pad 1 thru_hole circle (at -2.5 0 270) (size 1.5 1.5) (drill 1)
       (layers *.Cu *.Mask F.SilkS)
-      (net 76 N-0000029)
+      (net 78 N-0000093)
     )
     (pad 2 thru_hole circle (at 2.5 0 270) (size 1.5 1.5) (drill 1)
@@
     (pad 1 thru_hole circle (at -2.5 0 270) (size 1.5 1.5) (drill 1)
       (layers *.Cu *.Mask F.SilkS)
-      (net 73 N-00000100)
+      (net 76 N-0000086)
     )
     (pad 2 thru_hole circle (at 2.5 0 270) (size 1.5 1.5) (drill 1)
@@
     )
   )
+  (dimension 59.944 (width 0.3) (layer Dwgs.User)
+    (gr_text "59.944 mm" (at 308.816998 80.01 270) (layer Dwgs.User)
+      (effects (font (size 1.5 1.5) (thickness 0.3)))
+    )
+    (feature1 (pts (xy 299.974 109.982) (xy 310.166998 109.982)))
+    (feature2 (pts (xy 299.974 50.038) (xy 310.166998 50.038)))
+    (crossbar (pts (xy 307.466998 50.038) (xy 307.466998 109.982)))
+    (arrow1a (pts (xy 307.466998 109.982) (xy 306.880578 108.855497)))
+    (arrow1b (pts (xy 307.466998 109.982) (xy 308.053418 108.855497)))
+    (arrow2a (pts (xy 307.466998 50.038) (xy 306.880578 51.164503)))
+    (arrow2b (pts (xy 307.466998 50.038) (xy 308.053418 51.164503)))
+  )
+  (dimension 259.969 (width 0.3) (layer Dwgs.User)
+    (gr_text "259.969 mm" (at 169.9895 120.349005) (layer Dwgs.User)
+      (effects (font (size 1.5 1.5) (thickness 0.3)))
+    )
+    (feature1 (pts (xy 299.974 109.982) (xy 299.974 121.699005)))
+    (feature2 (pts (xy 40.005 109.982) (xy 40.005 121.699005)))
+    (crossbar (pts (xy 40.005 118.999005) (xy 299.974 118.999005)))
+    (arrow1a (pts (xy 299.974 118.999005) (xy 298.847497 119.585425)))
+    (arrow1b (pts (xy 299.974 118.999005) (xy 298.847497 118.412585)))
+    (arrow2a (pts (xy 40.005 118.999005) (xy 41.131503 119.585425)))
+    (arrow2b (pts (xy 40.005 118.999005) (xy 41.131503 118.412585)))
+  )
   (gr_text "SPI  20x2 #2" (at 195.6562 108.204) (layer F.SilkS)
     (effects (font (size 1.27 1.27) (thickness 0.254)))
@@
     (effects (font (size 1.27 1.27) (thickness 0.254)))
   )
-  (gr_text "4x 20mm Atmega328 Test Arena v0.3\nwww.iorodeo.com" (at 296.4942 85.4456 90) (layer F.SilkS)
+  (gr_text "4x 20mm Atmega328 Test Arena v0.3 R1\nwww.iorodeo.com" (at 296.4942 85.4456 90) (layer F.SilkS)
     (effects (font (size 1.016 1.016) (thickness 0.2032)))
   )
@@
   (segment (start 192.583 74.5555) (end 189.0275 71) (width 0.635) (layer F.Cu) (net 72))
   (segment (start 189.0275 71) (end 167.447 71) (width 0.635) (layer F.Cu) (net 72))
-  (segment (start 265.176 81.398) (end 265.176 76.08) (width 0.254) (layer B.Cu) (net 73))
-  (segment (start 265.278 81.5) (end 265.176 81.398) (width 0.254) (layer B.Cu) (net 73))
-  (segment (start 64.643 81.4238) (end 64.643 76.08) (width 0.254) (layer B.Cu) (net 74))
-  (segment (start 64.7192 81.5) (end 64.643 81.4238) (width 0.254) (layer B.Cu) (net 74))
-  (segment (start 241.681 82.8929) (end 241.681 83.7187) (width 0.254) (layer F.Cu) (net 75))
-  (segment (start 240.9066 84.6967) (end 240.9066 84.4931) (width 0.254) (layer F.Cu) (net 75))
-  (segment (start 241.3885 85.1786) (end 240.9066 84.6967) (width 0.254) (layer F.Cu) (net 75))
-  (segment (start 241.681 83.7187) (end 240.9066 84.4931) (width 0.254) (layer F.Cu) (net 75))
-  (segment (start 240.9066 84.4931) (end 236.6338 84.4931) (width 0.254) (layer F.Cu) (net 75))
-  (segment (start 241.3885 86.2584) (end 241.3885 85.1786) (width 0.254) (layer F.Cu) (net 75))
-  (segment (start 225.146 81.5) (end 225.146 76.08) (width 0.254) (layer B.Cu) (net 76))
-  (segment (start 104.775 81.424) (end 104.775 76.08) (width 0.254) (layer B.Cu) (net 77))
-  (segment (start 104.851 81.5) (end 104.775 81.424) (width 0.254) (layer B.Cu) (net 77))
-  (segment (start 144.907 81.449) (end 144.907 76.08) (width 0.254) (layer B.Cu) (net 78))
-  (segment (start 144.958 81.5) (end 144.907 81.449) (width 0.254) (layer B.Cu) (net 78))
-  (segment (start 184.963 81.5) (end 184.963 76.08) (width 0.254) (layer B.Cu) (net 79))
+  (segment (start 144.907 81.449) (end 144.907 76.08) (width 0.254) (layer B.Cu) (net 73))
+  (segment (start 144.958 81.5) (end 144.907 81.449) (width 0.254) (layer B.Cu) (net 73))
+  (segment (start 241.681 82.8929) (end 241.681 83.7187) (width 0.254) (layer F.Cu) (net 74))
+  (segment (start 240.9066 84.6967) (end 240.9066 84.4931) (width 0.254) (layer F.Cu) (net 74))
+  (segment (start 241.3885 85.1786) (end 240.9066 84.6967) (width 0.254) (layer F.Cu) (net 74))
+  (segment (start 241.681 83.7187) (end 240.9066 84.4931) (width 0.254) (layer F.Cu) (net 74))
+  (segment (start 240.9066 84.4931) (end 236.6338 84.4931) (width 0.254) (layer F.Cu) (net 74))
+  (segment (start 241.3885 86.2584) (end 241.3885 85.1786) (width 0.254) (layer F.Cu) (net 74))
+  (segment (start 64.643 81.4238) (end 64.643 76.08) (width 0.254) (layer B.Cu) (net 75))
+  (segment (start 64.7192 81.5) (end 64.643 81.4238) (width 0.254) (layer B.Cu) (net 75))
+  (segment (start 265.176 81.398) (end 265.176 76.08) (width 0.254) (layer B.Cu) (net 76))
+  (segment (start 265.278 81.5) (end 265.176 81.398) (width 0.254) (layer B.Cu) (net 76))
+  (segment (start 184.963 81.5) (end 184.963 76.08) (width 0.254) (layer B.Cu) (net 77))
+  (segment (start 225.146 81.5) (end 225.146 76.08) (width 0.254) (layer B.Cu) (net 78))
+  (segment (start 104.775 81.424) (end 104.775 76.08) (width 0.254) (layer B.Cu) (net 79))
+  (segment (start 104.851 81.5) (end 104.775 81.424) (width 0.254) (layer B.Cu) (net 79))
 )
