File: atmega328/four_panel/20mm_matrix/ver3/test_arena/arena.sch (KiCad schematic (older format))
At the start: 33 parts, among them P1 CONN15, P10 CONN_20X2, P2 CONN15, P3 CONN15, P4 CONN15, P5 CONN15, P6 CONN15, P7 CONN_20X2, P8 CONN_34X2, P9 CONN_2, Q1 MOSFET_NCHAN, SW1 SWITCH_INV, U1 SPARKFUN_TXB0104, U2 SPARKFUN_TXB0104, U3 SPARKFUN_TXB0104, U4 SPARKFUN_TXB0104, U5 SPARKFUN_TXB0104, U6 SPARKFUN_TXB0104, U7 SPARKFUN_TXB0104, U8 POLOLU_3V3

Commit message: Added gerber files for v0.3 of the g4 test arena.
Changed lines of the file:
@@
 Sheet 1 1
 Title ""
-Date "28 may 2015"
+Date "11 jun 2015"
 Rev ""
 Comp ""
@@
 Wire Wire Line
 	2000 4350 2000 4500
-$Comp
-L SPARKFUN_TXB0104 U1
-U 1 1 55662700
-P 1700 4000
-F 0 "U1" H 1700 3550 60  0000 C CNN
-F 1 "SPARKFUN_TXB0104" H 1700 4450 60  0000 C CNN
-F 2 "~" H 1650 4000 60  0000 C CNN
-F 3 "~" H 1650 4000 60  0000 C CNN
-	1    1700 4000
-	0    -1   -1   0
-$EndComp
-$Comp
-L SPARKFUN_TXB0104 U2
-U 1 1 5566270F
-P 3450 4000
-F 0 "U2" H 3450 3550 60  0000 C CNN
-F 1 "SPARKFUN_TXB0104" H 3450 4450 60  0000 C CNN
-F 2 "~" H 3400 4000 60  0000 C CNN
-F 3 "~" H 3400 4000 60  0000 C CNN
-	1    3450 4000
-	0    -1   -1   0
-$EndComp
-$Comp
-L SPARKFUN_TXB0104 U3
-U 1 1 55662728
-P 5200 4000
-F 0 "U3" H 5200 3550 60  0000 C CNN
-F 1 "SPARKFUN_TXB0104" H 5200 4450 60  0000 C CNN
-F 2 "~" H 5150 4000 60  0000 C CNN
-F 3 "~" H 5150 4000 60  0000 C CNN
-	1    5200 4000
-	0    -1   -1   0
-$EndComp
-$Comp
-L SPARKFUN_TXB0104 U4
-U 1 1 55662741
-P 6950 4000
-F 0 "U4" H 6950 3550 60  0000 C CNN
-F 1 "SPARKFUN_TXB0104" H 6950 4450 60  0000 C CNN
-F 2 "~" H 6900 4000 60  0000 C CNN
-F 3 "~" H 6900 4000 60  0000 C CNN
-	1    6950 4000
-	0    -1   -1   0
-$EndComp
-$Comp
-L SPARKFUN_TXB0104 U5
-U 1 1 5566275A
-P 8650 4000
-F 0 "U5" H 8650 3550 60  0000 C CNN
-F 1 "SPARKFUN_TXB0104" H 8650 4450 60  0000 C CNN
-F 2 "~" H 8600 4000 60  0000 C CNN
-F 3 "~" H 8600 4000 60  0000 C CNN
-	1    8650 4000
-	0    -1   -1   0
-$EndComp
-$Comp
-L SPARKFUN_TXB0104 U6
-U 1 1 55662773
-P 10300 4000
-F 0 "U6" H 10300 3550 60  0000 C CNN
-F 1 "SPARKFUN_TXB0104" H 10300 4450 60  0000 C CNN
-F 2 "~" H 10250 4000 60  0000 C CNN
-F 3 "~" H 10250 4000 60  0000 C CNN
-	1    10300 4000
-	0    -1   -1   0
-$EndComp
 Wire Wire Line
 	1500 4350 1500 4500
@@
 	1    2000 4500
 	1    0    0    -1
-$EndComp
-$Comp
-L SPARKFUN_TXB0104 U7
-U 1 1 55663A70
-P 6150 7650
-F 0 "U7" H 6150 7200 60  0000 C CNN
-F 1 "SPARKFUN_TXB0104" H 6150 8100 60  0000 C CNN
-F 2 "~" H 6100 7650 60  0000 C CNN
-F 3 "~" H 6100 7650 60  0000 C CNN
-	1    6150 7650
-	0    -1   -1   0
 $EndComp
 Text Label 1500 3500 1    60   ~ 0
@@
 NoConn ~ 6250 7300
 NoConn ~ 6250 8000
+$Comp
+L PWR_FLAG #FLG034
+U 1 1 557A1B99
+P 850 13150
+F 0 "#FLG034" H 850 13245 30  0001 C CNN
+F 1 "PWR_FLAG" H 850 13330 30  0000 C CNN
+F 2 "" H 850 13150 60  0000 C CNN
+F 3 "" H 850 13150 60  0000 C CNN
+	1    850  13150
+	1    0    0    -1
+$EndComp
+Wire Wire Line
+	850  13150 850  13300
+Text Label 850  13300 3    60   ~ 0
+5V
+$Comp
+L SPARKFUN_TXB0104 U1
+U 1 1 557A20EF
+P 1700 4000
+F 0 "U1" H 1700 4450 60  0000 C CNN
+F 1 "SPARKFUN_TXB0104" H 1700 3400 60  0000 C CNN
+F 2 "~" H 1650 4000 60  0000 C CNN
+F 3 "~" H 1650 4000 60  0000 C CNN
+	1    1700 4000
+	0    -1   -1   0
+$EndComp
+$Comp
+L SPARKFUN_TXB0104 U2
+U 1 1 557A20FE
+P 3450 4000
+F 0 "U2" H 3450 4450 60  0000 C CNN
+F 1 "SPARKFUN_TXB0104" H 3450 3450 60  0000 C CNN
+F 2 "~" H 3400 4000 60  0000 C CNN
+F 3 "~" H 3400 4000 60  0000 C CNN
+	1    3450 4000
+	0    -1   -1   0
+$EndComp
+$Comp
+L SPARKFUN_TXB0104 U3
+U 1 1 557A210D
+P 5200 4000
+F 0 "U3" H 5200 4450 60  0000 C CNN
+F 1 "SPARKFUN_TXB0104" H 5200 3450 60  0000 C CNN
+F 2 "~" H 5150 4000 60  0000 C CNN
+F 3 "~" H 5150 4000 60  0000 C CNN
+	1    5200 4000
+	0    -1   -1   0
+$EndComp
+$Comp
+L SPARKFUN_TXB0104 U4
+U 1 1 557A211C
+P 6950 4000
+F 0 "U4" H 6950 4450 60  0000 C CNN
+F 1 "SPARKFUN_TXB0104" H 6950 3450 60  0000 C CNN
+F 2 "~" H 6900 4000 60  0000 C CNN
+F 3 "~" H 6900 4000 60  0000 C CNN
+	1    6950 4000
+	0    -1   -1   0
+$EndComp
+$Comp
+L SPARKFUN_TXB0104 U5
+U 1 1 557A212B
+P 8650 4000
+F 0 "U5" H 8650 4450 60  0000 C CNN
+F 1 "SPARKFUN_TXB0104" H 8650 3450 60  0000 C CNN
+F 2 "~" H 8600 4000 60  0000 C CNN
+F 3 "~" H 8600 4000 60  0000 C CNN
+	1    8650 4000
+	0    -1   -1   0
+$EndComp
+$Comp
+L SPARKFUN_TXB0104 U6
+U 1 1 557A213A
+P 10300 4000
+F 0 "U6" H 10300 4450 60  0000 C CNN
+F 1 "SPARKFUN_TXB0104" H 10300 3450 60  0000 C CNN
+F 2 "~" H 10250 4000 60  0000 C CNN
+F 3 "~" H 10250 4000 60  0000 C CNN
+	1    10300 4000
+	0    -1   -1   0
+$EndComp
+$Comp
+L SPARKFUN_TXB0104 U7
+U 1 1 557A2149
+P 6150 7650
+F 0 "U7" H 6150 8100 60  0000 C CNN
+F 1 "SPARKFUN_TXB0104" H 6100 7050 60  0000 C CNN
+F 2 "~" H 6100 7650 60  0000 C CNN
+F 3 "~" H 6100 7650 60  0000 C CNN
+	1    6150 7650
+	0    -1   -1   0
+$EndComp
 $EndSCHEMATC
