File: atmega328/four_panel/20mm_matrix/ver3/12_18_arena/arena.kicad_pcb (KiCad board)
At the start: 2 copper layers, 85 parts, among them P1 CONN15, P10 CONN15, P11 CONN15, P12 CONN15, P13 CONN_2, P14 CONN_2, P15 CONN_2, P16 CONN_2, P17 CONN_2, P18 CONN_2, P19 CONN_2, P2 CONN15, P20 CONN_2, P21 CONN_2, P22 CONN_2, P23 CONN_2, P24 CONN_2, P25 CONN_34X2, P26 CONN_2, P3 CONN15, P4 CONN15, P5 CONN15, P6 CONN15, P7 CONN15, P8 CONN15, P9 CONN15, Q1 MOSFET_NCHAN, SW1 SWITCH_INV, U1 SPARKFUN_TXB0104, U10 SPARKFUN_TXB0104, U11 SPARKFUN_TXB0104, U12 SPARKFUN_TXB0104, U13 POLOLU_3V3, U2 SPARKFUN_TXB0104, U3 SPARKFUN_TXB0104, U4 SPARKFUN_TXB0104, U5 SPARKFUN_TXB0104, U6 SPARKFUN_TXB0104, U7 SPARKFUN_TXB0104, U8 SPARKFUN_TXB0104, U9 SPARKFUN_TXB0104

Commit message: Worked on 12-18 arena layout.
Parts:
- moved P25 333.7 mm to (327.5, 63.6), turned to 180 degrees
- moved C18 259.8 mm to (50.9, 254.8), turned to 180 degrees
- moved P26 112.4 mm to (92.2, 64.2)
- moved U13 110.0 mm to (70.9, 84.1)
- moved SW1 98.2 mm to (69.5, 69.4)
- moved U6 25.4 mm to (176.7, 78.4)
- moved U7 25.4 mm to (229.7, 78.4)
- moved R6 25.4 mm to (174.1, 93.0)
- moved P4 25.4 mm to (104.1, 145.4)
- moved P9 25.4 mm to (302.3, 145.4)
- moved P10 25.4 mm to (324.8, 184.3)
- moved P3 25.4 mm to (81.6, 184.3)
- moved P16 25.4 mm to (97.0, 139.5)
- moved P21 25.4 mm to (309.4, 139.5)
- moved R10 25.4 mm to (331.7, 176.4)
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Other:
- board outline added: 330.2 x 237.7 mm

Commit message: Arena modifications.
Parts:
- moved R24 451.2 mm to (0.00, 0.00), turned to 0 degrees
- moved U12 446.0 mm to (0.00, 0.00), turned to 0 degrees
- moved C12 435.0 mm to (0.00, 0.00), turned to 0 degrees
- moved P24 432.8 mm to (0.00, 0.00), turned to 0 degrees
- moved R23 431.3 mm to (0.00, 0.00)
- moved R12 431.2 mm to (0.00, 0.00), turned to 0 degrees
- moved P12 424.2 mm to (0.00, 0.00), turned to 0 degrees
- moved U11 422.9 mm to (0.00, 0.00), turned to 0 degrees
- moved C11 414.8 mm to (0.00, 0.00)
- moved P23 411.2 mm to (0.00, 0.00), turned to 0 degrees
- moved R11 408.4 mm to (0.00, 0.00)
- moved P11 403.6 mm to (0.00, 0.00), turned to 0 degrees
- moved R22 400.2 mm to (0.00, 0.00), turned to 0 degrees
- moved U10 388.9 mm to (0.00, 0.00), turned to 0 degrees
- moved C10 384.3 mm to (0.00, 0.00), turned to 0 degrees
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Other:
- board outline removed

Commit message: Finished pre-routing layout.
Parts:
- added C19: 10uF, Capacitor_Polarized, F.Cu at (255.4, 85.2)
- added C20: 10uF, Capacitor_Polarized, F.Cu at (301.3, 111.7)
- added C21: 10uF, Capacitor_Polarized, F.Cu at (335.3, 152.3)
- added C22: 10uF, Capacitor_Polarized, F.Cu at (353.4, 202.1)
- added C23: 10uF, Capacitor_Polarized, F.Cu at (353.4, 255.1)
- added P27: CONN_2, TERM_7P5MM, F.Cu at (106.7, 67.3)
- added P28: CONN_1, 0P25_MOUNT_HOLE, F.Cu at (76.2, 91.4)
- added P29: CONN_1, 0P25_MOUNT_HOLE, F.Cu at (330.2, 91.4)
- added P30: CONN_1, 0P25_MOUNT_HOLE, F.Cu at (330.2, 294.6)
- added P31: CONN_1, 0P25_MOUNT_HOLE, F.Cu at (76.2, 294.6)
- C18: value CP -> 10uf
- moved R24 454.9 mm to (345.4, 295.9), turned to 160 degrees
- moved U12 446.0 mm to (346.6, 280.8), turned to 160 degrees
- moved C12 435.0 mm to (331.3, 282.0), turned to 340 degrees
- moved P24 432.8 mm to (333.4, 276.0), turned to 160 degrees
- moved R23 431.3 mm to (355.8, 243.8)
- moved R12 431.2 mm to (335.2, 271.2), turned to 340 degrees
- moved P12 424.2 mm to (324.8, 272.9), turned to 250 degrees
- moved U11 422.9 mm to (355.8, 228.6), turned to 180 degrees
- moved C11 414.8 mm to (341.8, 234.9)
- moved P23 411.2 mm to (341.8, 228.6), turned to 180 degrees
- moved R11 408.4 mm to (341.8, 223.5)
- moved P11 403.6 mm to (332.6, 228.6), turned to 270 degrees
- moved R22 400.2 mm to (351.8, 190.7), turned to 20 degrees
- moved U10 388.9 mm to (346.6, 176.4), turned to 200 degrees
- moved C10 384.3 mm to (335.6, 187.2), turned to 20 degrees
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Connections:
- C8 pad 2: (no net) -> GND
Other:
- board outline added: 330.2 x 238.5 mm
- net class 3V3Pwr added: clearance 0.254, trace_width 0.635, via_dia 0.889, via_drill 0.635
- net class Pwr: trace_width 0.635 -> 1.524
- board text added: "+5V"
- board text added: "GND"

Commit message: Finished design of 12-18 arena. Routed and created gerber files.`
Routing:
- net GND: track 0.00 -> 1346.9 mm
- net /5V: track 0.00 -> 980.7 mm
- net /3V3: track 0.00 -> 700.4 mm, vias 0 -> 2
- net /EXT_INT_5V: track 0.00 -> 613.7 mm, vias 0 -> 1
- net /CS_6_5V: track 0.00 -> 608.4 mm
- net /CS_1_5V: track 0.00 -> 586.9 mm
- net /RESET_PAN: track 0.00 -> 586.1 mm, vias 0 -> 4
- net /CS_5_5V: track 0.00 -> 584.5 mm, vias 0 -> 2
- net /CS_2_5V: track 0.00 -> 581.9 mm
- net /CS_4_5V: track 0.00 -> 577.6 mm
- net /CS_7_5V: track 0.00 -> 568.6 mm, vias 0 -> 5
- net /CS_0_5V: track 0.00 -> 564.8 mm, vias 0 -> 2
- net /CS_3_5V: track 0.00 -> 561.4 mm
- net /CS_0_3V3: track 0.00 -> 477.2 mm
- net /CS_1_3V3: track 0.00 -> 464.9 mm, vias 0 -> 2
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Other:
- net class Pwr: trace_width 1.524 -> 0.635

Commit message: Added #4 ground holes.
Parts:
- added P32: CONN_1, #4_THROUGH_HOLE, F.Cu at (364.7, 67.1)
- added P33: CONN_1, #4_THROUGH_HOLE, F.Cu at (41.7, 298.4)
- added P34: CONN_1, #4_THROUGH_HOLE, F.Cu at (364.7, 298.4)
- added P35: CONN_1, #4_THROUGH_HOLE, F.Cu at (41.7, 67.1)
Routing:
- net GND: track 1346.9 -> 1478.8 mm, vias 0 -> 1
Other:
- net class Pwr: trace_width 0.635 -> 1.524
- board text added: "+5V (CENT POS)"

Commit message: Added .zip of gerber files.
Other:
- board text added: "12-18 Panels G4 Arena v0.1 R1 www.iorodeo.com"
Changed lines of the file:
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@@
     (links 378)
     (no_connects 0)
-    (area 37.949999 63.349999 368.450001 302.121564)
+    (area 37.949999 61.4464 388.698276 326.804008)
     (thickness 1.6)
-    (drawings 15)
+    (drawings 18)
     (tracks 2212)
     (zones 0)
@@
     )
   )
+  (gr_text "12-18 Panels G4 Arena v0.1 R1\nwww.iorodeo.com" (at 41.402 110.49 90) (layer F.SilkS)
+    (effects (font (size 1.5 1.5) (thickness 0.3)))
+  )
+  (dimension 238.506 (width 0.3) (layer Dwgs.User)
+    (gr_text "238.506 mm" (at 381.33399 182.753001 270) (layer Dwgs.User)
+      (effects (font (size 1.5 1.5) (thickness 0.3)))
+    )
+    (feature1 (pts (xy 368.3 302.006) (xy 382.68399 302.006001)))
+    (feature2 (pts (xy 368.3 63.5) (xy 382.68399 63.500001)))
+    (crossbar (pts (xy 379.98399 63.500001) (xy 379.98399 302.006001)))
+    (arrow1a (pts (xy 379.98399 302.006001) (xy 379.39757 300.879498)))
+    (arrow1b (pts (xy 379.98399 302.006001) (xy 380.57041 300.879498)))
+    (arrow2a (pts (xy 379.98399 63.500001) (xy 379.39757 64.626504)))
+    (arrow2b (pts (xy 379.98399 63.500001) (xy 380.57041 64.626504)))
+  )
+  (dimension 330.2 (width 0.3) (layer Dwgs.User)
+    (gr_text "330.200 mm" (at 203.2 325.454007) (layer Dwgs.User)
+      (effects (font (size 1.5 1.5) (thickness 0.3)))
+    )
+    (feature1 (pts (xy 368.3 302.006) (xy 368.3 326.804007)))
+    (feature2 (pts (xy 38.1 302.006) (xy 38.1 326.804007)))
+    (crossbar (pts (xy 38.1 324.104007) (xy 368.3 324.104007)))
+    (arrow1a (pts (xy 368.3 324.104007) (xy 367.173497 324.690427)))
+    (arrow1b (pts (xy 368.3 324.104007) (xy 367.173497 323.517587)))
+    (arrow2a (pts (xy 38.1 324.104007) (xy 39.226503 324.690427)))
+    (arrow2b (pts (xy 38.1 324.104007) (xy 39.226503 323.517587)))
+  )
   (gr_text "+5V (CENT POS)" (at 82.042 80.264) (layer F.SilkS)
     (effects (font (size 1.524 1.524) (thickness 0.3048)))
@@
   (segment (start 321.0333 175.0745) (end 321.0333 179.2476) (width 0.254) (layer F.Cu) (net 89))
   (segment (start 321.3081 174.7997) (end 321.0333 175.0745) (width 0.254) (layer F.Cu) (net 89))
-  (segment (start 319.063464 121.43138) (end 319.063464 121.118536) (width 1.524) (layer B.Cu) (net 90) (status C00000))
+  (segment (start 319.063464 121.43138) (end 319.063464 121.118536) (width 1.524) (layer B.Cu) (net 90))
   (segment (start 340.868 82.55) (end 340.868 80.772) (width 1.524) (layer F.Cu) (net 90))
   (segment (start 340.868 84.582) (end 340.868 82.55) (width 1.524) (layer F.Cu) (net 90))
   (via (at 340.868 84.582) (size 0.889) (layers F.Cu B.Cu) (net 90))
   (segment (start 340.868 99.314) (end 340.868 84.582) (width 1.524) (layer B.Cu) (net 90))
-  (segment (start 319.063464 121.118536) (end 340.868 99.314) (width 1.524) (layer B.Cu) (net 90) (status 400000))
+  (segment (start 319.063464 121.118536) (end 340.868 99.314) (width 1.524) (layer B.Cu) (net 90))
   (segment (start 340.868 80.772) (end 340.868 81.28) (width 1.524) (layer F.Cu) (net 90))
   (segment (start 340.868 81.28) (end 340.868 80.772) (width 1.524) (layer F.Cu) (net 90))

Commit message: Added new version of 12-18 arena.
Parts:
- removed U1, U10, U11, U12, U2, U3, U4, U5, U6, U7, U8, U9: SPARKFUN_TXB0104, SPARKFUN_TXB0104
- removed U13: POLOLU_3V3, POLOLU_3V3
- added C24: 30pF, C1, F.Cu at (46.4, 245.7)
- added C25: 30pF, C1, F.Cu at (221.0, 72.4)
- added C26: 30pF, C1, F.Cu at (358.1, 210.8)
- added C27: 30pF, C1, F.Cu at (46.4, 240.7)
- added C28: 30pF, C1, F.Cu at (226.1, 72.4)
- added C29: 30pF, C1, F.Cu at (358.1, 215.9)
- added C30: 30pF, C1, F.Cu at (46.4, 235.6)
- added C31: 30pF, C1, F.Cu at (231.1, 72.4)
- added C32: 30pF, C1, F.Cu at (358.1, 221.0)
- added C33: 30pF, C1, F.Cu at (46.4, 230.5)
- added C34: 30pF, C1, F.Cu at (236.2, 72.4)
- added C35: 30pF, C1, F.Cu at (358.1, 226.1)
- added C36: 30pF, C1, F.Cu at (46.4, 225.4)
- added C37: 30pF, C1, F.Cu at (241.3, 72.4)
- added C38: 30pF, C1, F.Cu at (358.1, 231.1)
- added C39: 30pF, C1, F.Cu at (46.4, 220.3)
- added C40: 30pF, C1, F.Cu at (246.4, 72.4)
- added C41: 30pF, C1, F.Cu at (358.1, 236.2)
- added C42: 30pF, C1, F.Cu at (46.4, 215.3)
- added C43: 30pF, C1, F.Cu at (251.5, 72.4)
- added C44: 30pF, C1, F.Cu at (358.1, 241.3)
- added C45: 30pF, C1, F.Cu at (46.4, 210.2)
- added C46: 30pF, C1, F.Cu at (256.5, 72.4)
- added C47: 30pF, C1, F.Cu at (358.1, 246.4)
- moved R24 15.4 mm to (339.6, 281.7), turned to 250 degrees
- moved R17 14.6 mm to (132.1, 101.1), turned to 30 degrees
- moved R21 14.5 mm to (316.5, 136.7), turned to 310 degrees
- moved R16 14.4 mm to (92.7, 132.8), turned to 50 degrees
- moved R23 14.3 mm to (349.2, 231.1), turned to 270 degrees
- moved R22 14.2 mm to (341.4, 181.1), turned to 290 degrees
- moved R18 14.1 mm to (180.3, 84.1), turned to 10 degrees
- moved R14 14.0 mm to (57.1, 225.8), turned to 90 degrees
- moved R13 14.0 mm to (65.0, 275.8), turned to 110 degrees
- moved R19 13.9 mm to (231.4, 85.1), turned to 350 degrees
- moved R20 13.8 mm to (278.9, 103.1), turned to 330 degrees
- moved R15 13.8 mm to (66.8, 175.8), turned to 70 degrees
- moved Q1 10.8 mm to (344.8, 120.0)
- moved R26 10.8 mm to (344.8, 112.4)
- moved R25 10.8 mm to (349.9, 116.2)
Connections:
- net /MISO_0_3V3 renamed /MISO_0
- net /MISO_0_5V renamed /_MISO_0
- net /MISO_10_3V3 renamed /MISO_10
- net /MISO_10_5V renamed /_MISO_10
- net /MISO_11_3V3 renamed /MISO_11
- net /MISO_11_5V renamed /_MISO_11
- net /MISO_1_3V3 renamed /MISO_1
- net /MISO_1_5V renamed /_MISO_1
- net /MISO_2_3V3 renamed /MISO_2
- net /MISO_2_5V renamed /_MISO_2
- net /MISO_3_3V3 renamed /MISO_3
- net /MISO_3_5V renamed /_MISO_3
- net /MISO_4_3V3 renamed /MISO_4
- net /MISO_4_5V renamed /_MISO_4
- net /MISO_5_3V3 renamed /MISO_5
- net /MISO_5_5V renamed /_MISO_5
- net /MISO_6_3V3 renamed /MISO_6
- net /MISO_6_5V renamed /_MISO_6
- net /MISO_7_3V3 renamed /MISO_7
- net /MISO_7_5V renamed /_MISO_7
- net /MISO_8_3V3 renamed /MISO_8
- net /MISO_8_5V renamed /_MISO_8
- net /MISO_9_3V3 renamed /MISO_9
- net /MISO_9_5V renamed /_MISO_9
- P1 pad 10: /CS_3_5V -> /CS_3
- P1 pad 11: /CS_4_5V -> /CS_4
- P1 pad 12: /CS_5_5V -> /CS_5
- P1 pad 13: /CS_6_5V -> /CS_6
- P1 pad 14: /CS_7_5V -> /CS_7
- P1 pad 15: /EXT_INT_5V -> /EXT_INT
- P1 pad 4: /SCK_0_5V -> /SCK_0
- P1 pad 5: /MOSI_0_5V -> /MOSI_0
- P1 pad 7: /CS_0_5V -> /CS_0
- P1 pad 8: /CS_1_5V -> /CS_1
- P1 pad 9: /CS_2_5V -> /CS_2
- P10 pad 10: /CS_3_5V -> /CS_3
- P10 pad 11: /CS_4_5V -> /CS_4
- P10 pad 12: /CS_5_5V -> /CS_5
- P10 pad 13: /CS_6_5V -> /CS_6
- P10 pad 14: /CS_7_5V -> /CS_7
- P10 pad 15: /EXT_INT_5V -> /EXT_INT
- P10 pad 4: /SCK_9_5V -> /SCK_3
- P10 pad 5: /MOSI_9_5V -> /MOSI_9
- P10 pad 7: /CS_0_5V -> /CS_0
- P10 pad 8: /CS_1_5V -> /CS_1
- P10 pad 9: /CS_2_5V -> /CS_2
- P11 pad 10: /CS_3_5V -> /CS_3
- P11 pad 11: /CS_4_5V -> /CS_4
- P11 pad 12: /CS_5_5V -> /CS_5
- P11 pad 13: /CS_6_5V -> /CS_6
- P11 pad 14: /CS_7_5V -> /CS_7
- P11 pad 15: /EXT_INT_5V -> /EXT_INT
- P11 pad 4: /SCK_10_5V -> /SCK_4
- P11 pad 5: /MOSI_10_5V -> /MOSI_10
- P11 pad 7: /CS_0_5V -> /CS_0
- P11 pad 8: /CS_1_5V -> /CS_1
- P11 pad 9: /CS_2_5V -> /CS_2
- P12 pad 10: /CS_3_5V -> /CS_3
- P12 pad 11: /CS_4_5V -> /CS_4
- P12 pad 12: /CS_5_5V -> /CS_5
- P12 pad 13: /CS_6_5V -> /CS_6
- P12 pad 14: /CS_7_5V -> /CS_7
- P12 pad 15: /EXT_INT_5V -> /EXT_INT
- P12 pad 4: /SCK_11_5V -> /SCK_5
- P12 pad 5: /MOSI_11_5V -> /MOSI_11
- P12 pad 7: /CS_0_5V -> /CS_0
- P12 pad 8: /CS_1_5V -> /CS_1
- P12 pad 9: /CS_2_5V -> /CS_2
- P13 pad 1: N-0000073 -> N-0000044
- P14 pad 1: N-0000072 -> N-0000043
- P15 pad 1: N-0000071 -> N-0000042
- P16 pad 1: N-0000070 -> N-0000041
- P17 pad 1: N-0000068 -> N-0000040
- P18 pad 1: N-0000067 -> N-0000039
- P19 pad 1: N-0000066 -> N-0000038
- P2 pad 10: /CS_3_5V -> /CS_3
- P2 pad 11: /CS_4_5V -> /CS_4
- P2 pad 12: /CS_5_5V -> /CS_5
- P2 pad 13: /CS_6_5V -> /CS_6
- P2 pad 14: /CS_7_5V -> /CS_7
- P2 pad 15: /EXT_INT_5V -> /EXT_INT
- P2 pad 4: /SCK_1_5V -> /SCK_1
- P2 pad 5: /MOSI_1_5V -> /MOSI_1
- P2 pad 7: /CS_0_5V -> /CS_0
- P2 pad 8: /CS_1_5V -> /CS_1
- P2 pad 9: /CS_2_5V -> /CS_2
- P20 pad 1: N-0000065 -> N-0000030
- P21 pad 1: N-0000064 -> N-0000036
- P22 pad 1: N-0000063 -> N-0000033
- P23 pad 1: N-0000079 -> N-0000021
- P24 pad 1: N-0000081 -> N-0000020
- P25 pad 29: /MOSI_7_3V3 -> /MOSI_7
- P25 pad 30: /MOSI_8_3V3 -> /MOSI_8
- P25 pad 31: /MOSI_9_3V3 -> /MOSI_9
- P25 pad 32: /MOSI_10_3V3 -> /MOSI_10
- P25 pad 33: /MOSI_11_3V3 -> /MOSI_11
- P25 pad 35: /CS_0_3V3 -> /CS_0
- P25 pad 36: /CS_1_3V3 -> /CS_1
- P25 pad 37: /CS_2_3V3 -> /CS_2
- P25 pad 38: /CS_3_3V3 -> /CS_3
- P25 pad 39: /CS_4_3V3 -> /CS_4
- P25 pad 40: /CS_5_3V3 -> /CS_5
- P25 pad 41: /CS_6_3V3 -> /CS_6
- P25 pad 42: /CS_7_3V3 -> /CS_7
- P25 pad 43: /SCK_0_3V3 -> /SCK_0
- P25 pad 44: /SCK_1_3V3 -> /SCK_1
- P25 pad 45: /SCK_2_3V3 -> /SCK_2
- P25 pad 46: /SCK_3_3V3 -> /SCK_3
- P25 pad 47: /SCK_4_3V3 -> /SCK_4
- P25 pad 48: /SCK_5_3V3 -> /SCK_5
- P25 pad 49: /MOSI_0_3V3 -> /MOSI_0
- P25 pad 51: /MOSI_1_3V3 -> /MOSI_1
- P25 pad 53: /MOSI_2_3V3 -> /MOSI_2
- P25 pad 55: /MOSI_3_3V3 -> /MOSI_3
- P25 pad 57: /MOSI_4_3V3 -> /MOSI_4
- P25 pad 59: /MOSI_5_3V3 -> /MOSI_5
- P25 pad 61: /MOSI_6_3V3 -> /MOSI_6
- P25 pad 68: /EXT_INT_3V3 -> /EXT_INT
- P3 pad 10: /CS_3_5V -> /CS_3
- P3 pad 11: /CS_4_5V -> /CS_4
- P3 pad 12: /CS_5_5V -> /CS_5
- P3 pad 13: /CS_6_5V -> /CS_6
- P3 pad 14: /CS_7_5V -> /CS_7
- P3 pad 15: /EXT_INT_5V -> /EXT_INT
- P3 pad 4: /SCK_2_5V -> /SCK_2
- P3 pad 5: /MOSI_2_5V -> /MOSI_2
- P3 pad 7: /CS_0_5V -> /CS_0
- P3 pad 8: /CS_1_5V -> /CS_1
- P3 pad 9: /CS_2_5V -> /CS_2
- P4 pad 10: /CS_3_5V -> /CS_3
- P4 pad 11: /CS_4_5V -> /CS_4
- P4 pad 12: /CS_5_5V -> /CS_5
- P4 pad 13: /CS_6_5V -> /CS_6
- P4 pad 14: /CS_7_5V -> /CS_7
- P4 pad 15: /EXT_INT_5V -> /EXT_INT
- P4 pad 4: /SCK_3_5V -> /SCK_3
- P4 pad 5: /MOSI_3_5V -> /MOSI_3
- P4 pad 7: /CS_0_5V -> /CS_0
- P4 pad 8: /CS_1_5V -> /CS_1
- P4 pad 9: /CS_2_5V -> /CS_2
- P5 pad 10: /CS_3_5V -> /CS_3
- P5 pad 11: /CS_4_5V -> /CS_4
- P5 pad 12: /CS_5_5V -> /CS_5
- P5 pad 13: /CS_6_5V -> /CS_6
- P5 pad 14: /CS_7_5V -> /CS_7
- P5 pad 15: /EXT_INT_5V -> /EXT_INT
- P5 pad 4: /SCK_4_5V -> /SCK_4
- P5 pad 5: /MOSI_4_5V -> /MOSI_4
- P5 pad 7: /CS_0_5V -> /CS_0
- P5 pad 8: /CS_1_5V -> /CS_1
- P5 pad 9: /CS_2_5V -> /CS_2
- P6 pad 10: /CS_3_5V -> /CS_3
- P6 pad 11: /CS_4_5V -> /CS_4
- P6 pad 12: /CS_5_5V -> /CS_5
- P6 pad 13: /CS_6_5V -> /CS_6
- P6 pad 14: /CS_7_5V -> /CS_7
- P6 pad 15: /EXT_INT_5V -> /EXT_INT
- P6 pad 4: /SCK_5_5V -> /SCK_5
- P6 pad 5: /MOSI_5_5V -> /MOSI_5
- P6 pad 7: /CS_0_5V -> /CS_0
- P6 pad 8: /CS_1_5V -> /CS_1
- P6 pad 9: /CS_2_5V -> /CS_2
- P7 pad 10: /CS_3_5V -> /CS_3
- P7 pad 11: /CS_4_5V -> /CS_4
- P7 pad 12: /CS_5_5V -> /CS_5
- P7 pad 13: /CS_6_5V -> /CS_6
- P7 pad 14: /CS_7_5V -> /CS_7
- P7 pad 15: /EXT_INT_5V -> /EXT_INT
- P7 pad 4: /SCK_6_5V -> /SCK_0
- P7 pad 5: /MOSI_6_5V -> /MOSI_6
- P7 pad 7: /CS_0_5V -> /CS_0
- P7 pad 8: /CS_1_5V -> /CS_1
- P7 pad 9: /CS_2_5V -> /CS_2
- P8 pad 10: /CS_3_5V -> /CS_3
- P8 pad 11: /CS_4_5V -> /CS_4
- P8 pad 12: /CS_5_5V -> /CS_5
- P8 pad 13: /CS_6_5V -> /CS_6
- P8 pad 14: /CS_7_5V -> /CS_7
- P8 pad 15: /EXT_INT_5V -> /EXT_INT
- P8 pad 4: /SCK_7_5V -> /SCK_1
- P8 pad 5: /MOSI_7_5V -> /MOSI_7
- P8 pad 7: /CS_0_5V -> /CS_0
- P8 pad 8: /CS_1_5V -> /CS_1
- P8 pad 9: /CS_2_5V -> /CS_2
- P9 pad 10: /CS_3_5V -> /CS_3
- P9 pad 11: /CS_4_5V -> /CS_4
- P9 pad 12: /CS_5_5V -> /CS_5
- P9 pad 13: /CS_6_5V -> /CS_6
- P9 pad 14: /CS_7_5V -> /CS_7
- P9 pad 15: /EXT_INT_5V -> /EXT_INT
- P9 pad 4: /SCK_8_5V -> /SCK_2
- P9 pad 5: /MOSI_8_5V -> /MOSI_8
- P9 pad 7: /CS_0_5V -> /CS_0
- P9 pad 8: /CS_1_5V -> /CS_1
- P9 pad 9: /CS_2_5V -> /CS_2
- R13 pad 1: N-00000182 -> N-0000044
- R14 pad 1: N-00000170 -> N-0000043
- R15 pad 1: N-00000169 -> N-0000042
- R16 pad 1: N-00000171 -> N-0000041
- R17 pad 1: N-00000175 -> N-0000040
- R18 pad 1: N-0000047 (its old number) -> N-0000039
- R19 pad 1: N-0000042 -> N-0000038
- R20 pad 1: N-0000057 (its old number) -> N-0000030
- R21 pad 1: N-000003 -> N-0000036
- R22 pad 1: N-0000026 -> N-0000033
- R23 pad 1: N-0000086 -> N-0000021
- R24 pad 1: N-00000102 -> N-0000020
Routing:
- net /CS_1: track 0.00 -> 804.0 mm
- net /CS_5: track 0.00 -> 761.4 mm
- net /CS_3: track 0.00 -> 757.9 mm, vias 0 -> 1
- net /CS_4: track 0.00 -> 749.6 mm, vias 0 -> 1
- net /CS_2: track 0.00 -> 743.3 mm, vias 0 -> 1
- net /CS_0: track 0.00 -> 742.6 mm, vias 0 -> 1
- net /CS_6: track 0.00 -> 735.6 mm
- net /CS_7: track 0.00 -> 732.6 mm, vias 0 -> 3
- net /3V3: track 700.4 -> 0.00 mm, vias 2 -> 0
- net /EXT_INT: track 0.00 -> 619.2 mm, vias 0 -> 2
- net /EXT_INT_5V: track 613.7 -> 0.00 mm, vias 1 -> 0
- net /CS_6_5V: track 608.4 -> 0.00 mm
- net /CS_1_5V: track 586.9 -> 0.00 mm
- net /CS_5_5V: track 584.5 -> 0.00 mm, vias 2 -> 0
- net /CS_2_5V: track 581.9 -> 0.00 mm
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
Commit message: Added keepout zones and re-routed 12-18 arena.
Routing:
- net /CS_6: track 735.6 -> 800.0 mm
- net /CS_2: track 743.3 -> 806.7 mm
- net /CS_0: track 742.6 -> 805.2 mm
- net /CS_4: track 749.6 -> 796.8 mm, vias 1 -> 2
- net /EXT_INT: track 619.2 -> 665.5 mm, vias 2 -> 1
- net /SCK_5: track 421.4 -> 386.3 mm, vias 0 -> 1
- net /MOSI_0: track 394.8 -> 416.5 mm
- net /CS_7: track 732.6 -> 754.3 mm, vias 3 -> 0
- net /MISO_0: track 417.8 -> 435.6 mm, vias 2 -> 0
- net /CS_1: track 804.0 -> 787.1 mm, vias 0 -> 1
- net /5V: track 908.2 -> 894.0 mm
- net /RESET_PAN: track 615.6 -> 629.8 mm, vias 1 -> 2
- net /MOSI_3: track 261.3 -> 274.0 mm, vias 2 -> 1
- net /SCK_3: track 378.9 -> 391.0 mm
- net /SCK_4: track 385.9 -> 397.8 mm, vias 2 -> 1
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Other:
- net class 3V3Pwr removed
