File: atmega328/four_panel/20mm_matrix/ver3/driver_w_leds/driver.sch (KiCad schematic (older format))
At the start: 308 parts, among them IC1 ATMEGA328P-M, IC2 ATMEGA328P-M, IC3 ATMEGA328P-M, IC4 ATMEGA328P-M, P1 CONN_2X2, P2 CONN_2X2, P3 CONN_2X2, P4 CONN_2X2, X1 CER_RESO, X2 CER_RESO, X3 CER_RESO, X4 CER_RESO

Commit message: Added high current (sink/source) unity gain buffers.
Parts:
- added U1, U10, U11, U12, U13, U14, U15, U16, U17, U18, U19, U2, U20, U21, U22, U23, U24, U25, U26, U27, U28, U29, U3, U30, U31, U32, U4, U5, U6, U7, U8, U9: DMC2400UV, ~, symbol DMC2400UV
Connections:
- net +5V: now also U1.4 (S2), U10.4 (S2), U11.4 (S2), U12.4 (S2), U13.4 (S2), U14.4 (S2), U15.4 (S2), U16.4 (S2), U17.4 (S2), U18.4 (S2), U19.4 (S2), U2.4 (S2), U20.4 (S2), U21.4 (S2), U22.4 (S2), U23.4 (S2), U24.4 (S2), U25.4 (S2), U26.4 (S2), U27.4 (S2), U28.4 (S2), U29.4 (S2), U3.4 (S2), U30.4 (S2), U31.4 (S2), U32.4 (S2), U4.4 (S2), U5.4 (S2), U6.4 (S2), U7.4 (S2), U8.4 (S2), U9.4 (S2)
- net GND: now also U1.1 (S1), U10.1 (S1), U11.1 (S1), U12.1 (S1), U13.1 (S1), U14.1 (S1), U15.1 (S1), U16.1 (S1), U17.1 (S1), U18.1 (S1), U19.1 (S1), U2.1 (S1), U20.1 (S1), U21.1 (S1), U22.1 (S1), U23.1 (S1), U24.1 (S1), U25.1 (S1), U26.1 (S1), U27.1 (S1), U28.1 (S1), U29.1 (S1), U3.1 (S1), U30.1 (S1), U31.1 (S1), U32.1 (S1), U4.1 (S1), U5.1 (S1), U6.1 (S1), U7.1 (S1), U8.1 (S1), U9.1 (S1)
- net ROW0_DRV0: now also U1.2 (G1), U1.5 (G2); no longer D1.2 (K), D17.2 (K), D25.2 (K), D33.2 (K), D41.2 (K), D49.2 (K), D57.2 (K), D9.2 (K)
- net ROW0_DRV1: now also U9.2 (G1), U9.5 (G2); no longer D105.2 (K), D113.2 (K), D121.2 (K), D65.2 (K), D73.2 (K), D81.2 (K), D89.2 (K), D97.2 (K)
- net ROW0_DRV2: now also U17.2 (G1), U17.5 (G2); no longer D129.2 (K), D137.2 (K), D145.2 (K), D153.2 (K), D161.2 (K), D169.2 (K), D177.2 (K), D185.2 (K)
- net ROW0_DRV3: now also U25.2 (G1), U25.5 (G2); no longer D193.2 (K), D201.2 (K), D209.2 (K), D217.2 (K), D225.2 (K), D233.2 (K), D241.2 (K), D249.2 (K)
- net ROW1_DRV0: now also U2.2 (G1), U2.5 (G2); no longer D10.2 (K), D18.2 (K), D2.2 (K), D26.2 (K), D34.2 (K), D42.2 (K), D50.2 (K), D58.2 (K)
- net ROW1_DRV1: now also U10.2 (G1), U10.5 (G2); no longer D106.2 (K), D114.2 (K), D122.2 (K), D66.2 (K), D74.2 (K), D82.2 (K), D90.2 (K), D98.2 (K)
- net ROW1_DRV2: now also U18.2 (G1), U18.5 (G2); no longer D130.2 (K), D138.2 (K), D146.2 (K), D154.2 (K), D162.2 (K), D170.2 (K), D178.2 (K), D186.2 (K)
- net ROW1_DRV3: now also U26.2 (G1), U26.5 (G2); no longer D194.2 (K), D202.2 (K), D210.2 (K), D218.2 (K), D226.2 (K), D234.2 (K), D242.2 (K), D250.2 (K)
- net ROW2_DRV0: now also U3.2 (G1), U3.5 (G2); no longer D11.2 (K), D19.2 (K), D27.2 (K), D3.2 (K), D35.2 (K), D43.2 (K), D51.2 (K), D59.2 (K)
- net ROW2_DRV1: now also U11.2 (G1), U11.5 (G2); no longer D107.2 (K), D115.2 (K), D123.2 (K), D67.2 (K), D75.2 (K), D83.2 (K), D91.2 (K), D99.2 (K)
- net ROW2_DRV2: now also U19.2 (G1), U19.5 (G2); no longer D131.2 (K), D139.2 (K), D147.2 (K), D155.2 (K), D163.2 (K), D171.2 (K), D179.2 (K), D187.2 (K)
- net ROW2_DRV3: now also U27.2 (G1), U27.5 (G2); no longer D195.2 (K), D203.2 (K), D211.2 (K), D219.2 (K), D227.2 (K), D235.2 (K), D243.2 (K), D251.2 (K)
- net ROW3_DRV0: now also U4.2 (G1), U4.5 (G2); no longer D12.2 (K), D20.2 (K), D28.2 (K), D36.2 (K), D4.2 (K), D44.2 (K), D52.2 (K), D60.2 (K)
- net ROW3_DRV1: now also U12.2 (G1), U12.5 (G2); no longer D100.2 (K), D108.2 (K), D116.2 (K), D124.2 (K), D68.2 (K), D76.2 (K), D84.2 (K), D92.2 (K)
- net ROW3_DRV2: now also U20.2 (G1), U20.5 (G2); no longer D132.2 (K), D140.2 (K), D148.2 (K), D156.2 (K), D164.2 (K), D172.2 (K), D180.2 (K), D188.2 (K)
- net ROW3_DRV3: now also U28.2 (G1), U28.5 (G2); no longer D196.2 (K), D204.2 (K), D212.2 (K), D220.2 (K), D228.2 (K), D236.2 (K), D244.2 (K), D252.2 (K)
- net ROW4_DRV0: now also U5.2 (G1), U5.5 (G2); no longer D13.2 (K), D21.2 (K), D29.2 (K), D37.2 (K), D45.2 (K), D5.2 (K), D53.2 (K), D61.2 (K)
- net ROW4_DRV1: now also U13.2 (G1), U13.5 (G2); no longer D101.2 (K), D109.2 (K), D117.2 (K), D125.2 (K), D69.2 (K), D77.2 (K), D85.2 (K), D93.2 (K)
- net ROW4_DRV2: now also U21.2 (G1), U21.5 (G2); no longer D133.2 (K), D141.2 (K), D149.2 (K), D157.2 (K), D165.2 (K), D173.2 (K), D181.2 (K), D189.2 (K)
- net ROW4_DRV3: now also U29.2 (G1), U29.5 (G2); no longer D197.2 (K), D205.2 (K), D213.2 (K), D221.2 (K), D229.2 (K), D237.2 (K), D245.2 (K), D253.2 (K)
- net ROW5_DRV0: now also U6.2 (G1), U6.5 (G2); no longer D14.2 (K), D22.2 (K), D30.2 (K), D38.2 (K), D46.2 (K), D54.2 (K), D6.2 (K), D62.2 (K)
- net ROW5_DRV1: now also U14.2 (G1), U14.5 (G2); no longer D102.2 (K), D110.2 (K), D118.2 (K), D126.2 (K), D70.2 (K), D78.2 (K), D86.2 (K), D94.2 (K)
- net ROW5_DRV2: now also U22.2 (G1), U22.5 (G2); no longer D134.2 (K), D142.2 (K), D150.2 (K), D158.2 (K), D166.2 (K), D174.2 (K), D182.2 (K), D190.2 (K)
- net ROW5_DRV3: now also U30.2 (G1), U30.5 (G2); no longer D198.2 (K), D206.2 (K), D214.2 (K), D222.2 (K), D230.2 (K), D238.2 (K), D246.2 (K), D254.2 (K)
- net ROW6_DRV0: now also U7.2 (G1), U7.5 (G2); no longer D15.2 (K), D23.2 (K), D31.2 (K), D39.2 (K), D47.2 (K), D55.2 (K), D63.2 (K), D7.2 (K)
- net ROW6_DRV1: now also U15.2 (G1), U15.5 (G2); no longer D103.2 (K), D111.2 (K), D119.2 (K), D127.2 (K), D71.2 (K), D79.2 (K), D87.2 (K), D95.2 (K)
- net ROW6_DRV2: now also U23.2 (G1), U23.5 (G2); no longer D135.2 (K), D143.2 (K), D151.2 (K), D159.2 (K), D167.2 (K), D175.2 (K), D183.2 (K), D191.2 (K)
- net ROW6_DRV3: now also U31.2 (G1), U31.5 (G2); no longer D199.2 (K), D207.2 (K), D215.2 (K), D223.2 (K), D231.2 (K), D239.2 (K), D247.2 (K), D255.2 (K)
- net ROW7_DRV0: now also U8.2 (G1), U8.5 (G2); no longer D16.2 (K), D24.2 (K), D32.2 (K), D40.2 (K), D48.2 (K), D56.2 (K), D64.2 (K), D8.2 (K)
- net ROW7_DRV1: now also U16.2 (G1), U16.5 (G2); no longer D104.2 (K), D112.2 (K), D120.2 (K), D128.2 (K), D72.2 (K), D80.2 (K), D88.2 (K), D96.2 (K)
- net ROW7_DRV2: now also U24.2 (G1), U24.5 (G2); no longer D136.2 (K), D144.2 (K), D152.2 (K), D160.2 (K), D168.2 (K), D176.2 (K), D184.2 (K), D192.2 (K)
- net ROW7_DRV3: now also U32.2 (G1), U32.5 (G2); no longer D200.2 (K), D208.2 (K), D216.2 (K), D224.2 (K), D232.2 (K), D240.2 (K), D248.2 (K), D256.2 (K)
- new net ROW0_INV0: D1.2 (K), D17.2 (K), D25.2 (K), D33.2 (K), D41.2 (K), D49.2 (K), D57.2 (K), D9.2 (K), U1.3 (D2), U1.6 (D1)
- new net ROW0_INV1: D105.2 (K), D113.2 (K), D121.2 (K), D65.2 (K), D73.2 (K), D81.2 (K), D89.2 (K), D97.2 (K), U9.3 (D2), U9.6 (D1)
- new net ROW0_INV2: D129.2 (K), D137.2 (K), D145.2 (K), D153.2 (K), D161.2 (K), D169.2 (K), D177.2 (K), D185.2 (K), U17.3 (D2), U17.6 (D1)
- new net ROW0_INV3: D193.2 (K), D201.2 (K), D209.2 (K), D217.2 (K), D225.2 (K), D233.2 (K), D241.2 (K), D249.2 (K), U25.3 (D2), U25.6 (D1)
- new net ROW1_INV0: D10.2 (K), D18.2 (K), D2.2 (K), D26.2 (K), D34.2 (K), D42.2 (K), D50.2 (K), D58.2 (K), U2.3 (D2), U2.6 (D1)
- new net ROW1_INV1: D106.2 (K), D114.2 (K), D122.2 (K), D66.2 (K), D74.2 (K), D82.2 (K), D90.2 (K), D98.2 (K), U10.3 (D2), U10.6 (D1)
- new net ROW1_INV2: D130.2 (K), D138.2 (K), D146.2 (K), D154.2 (K), D162.2 (K), D170.2 (K), D178.2 (K), D186.2 (K), U18.3 (D2), U18.6 (D1)
- new net ROW1_INV3: D194.2 (K), D202.2 (K), D210.2 (K), D218.2 (K), D226.2 (K), D234.2 (K), D242.2 (K), D250.2 (K), U26.3 (D2), U26.6 (D1)
- new net ROW2_INV0: D11.2 (K), D19.2 (K), D27.2 (K), D3.2 (K), D35.2 (K), D43.2 (K), D51.2 (K), D59.2 (K), U3.3 (D2), U3.6 (D1)
- new net ROW2_INV1: D107.2 (K), D115.2 (K), D123.2 (K), D67.2 (K), D75.2 (K), D83.2 (K), D91.2 (K), D99.2 (K), U11.3 (D2), U11.6 (D1)
- new net ROW2_INV2: D131.2 (K), D139.2 (K), D147.2 (K), D155.2 (K), D163.2 (K), D171.2 (K), D179.2 (K), D187.2 (K), U19.3 (D2), U19.6 (D1)
- new net ROW2_INV3: D195.2 (K), D203.2 (K), D211.2 (K), D219.2 (K), D227.2 (K), D235.2 (K), D243.2 (K), D251.2 (K), U27.3 (D2), U27.6 (D1)
- new net ROW3_INV0: D12.2 (K), D20.2 (K), D28.2 (K), D36.2 (K), D4.2 (K), D44.2 (K), D52.2 (K), D60.2 (K), U4.3 (D2), U4.6 (D1)
- new net ROW3_INV1: D100.2 (K), D108.2 (K), D116.2 (K), D124.2 (K), D68.2 (K), D76.2 (K), D84.2 (K), D92.2 (K), U12.3 (D2), U12.6 (D1)
- new net ROW3_INV2: D132.2 (K), D140.2 (K), D148.2 (K), D156.2 (K), D164.2 (K), D172.2 (K), D180.2 (K), D188.2 (K), U20.3 (D2), U20.6 (D1)
- new net ROW3_INV3: D196.2 (K), D204.2 (K), D212.2 (K), D220.2 (K), D228.2 (K), D236.2 (K), D244.2 (K), D252.2 (K), U28.3 (D2), U28.6 (D1)
- new net ROW4_INV0: D13.2 (K), D21.2 (K), D29.2 (K), D37.2 (K), D45.2 (K), D5.2 (K), D53.2 (K), D61.2 (K), U5.3 (D2), U5.6 (D1)
- new net ROW4_INV1: D101.2 (K), D109.2 (K), D117.2 (K), D125.2 (K), D69.2 (K), D77.2 (K), D85.2 (K), D93.2 (K), U13.3 (D2), U13.6 (D1)
- new net ROW4_INV2: D133.2 (K), D141.2 (K), D149.2 (K), D157.2 (K), D165.2 (K), D173.2 (K), D181.2 (K), D189.2 (K), U21.3 (D2), U21.6 (D1)
- new net ROW4_INV3: D197.2 (K), D205.2 (K), D213.2 (K), D221.2 (K), D229.2 (K), D237.2 (K), D245.2 (K), D253.2 (K), U29.3 (D2), U29.6 (D1)
- new net ROW5_INV0: D14.2 (K), D22.2 (K), D30.2 (K), D38.2 (K), D46.2 (K), D54.2 (K), D6.2 (K), D62.2 (K), U6.3 (D2), U6.6 (D1)
- new net ROW5_INV1: D102.2 (K), D110.2 (K), D118.2 (K), D126.2 (K), D70.2 (K), D78.2 (K), D86.2 (K), D94.2 (K), U14.3 (D2), U14.6 (D1)
- new net ROW5_INV2: D134.2 (K), D142.2 (K), D150.2 (K), D158.2 (K), D166.2 (K), D174.2 (K), D182.2 (K), D190.2 (K), U22.3 (D2), U22.6 (D1)
- new net ROW5_INV3: D198.2 (K), D206.2 (K), D214.2 (K), D222.2 (K), D230.2 (K), D238.2 (K), D246.2 (K), D254.2 (K), U30.3 (D2), U30.6 (D1)
- new net ROW6_INV0: D15.2 (K), D23.2 (K), D31.2 (K), D39.2 (K), D47.2 (K), D55.2 (K), D63.2 (K), D7.2 (K), U7.3 (D2), U7.6 (D1)
- new net ROW6_INV1: D103.2 (K), D111.2 (K), D119.2 (K), D127.2 (K), D71.2 (K), D79.2 (K), D87.2 (K), D95.2 (K), U15.3 (D2), U15.6 (D1)
- new net ROW6_INV2: D135.2 (K), D143.2 (K), D151.2 (K), D159.2 (K), D167.2 (K), D175.2 (K), D183.2 (K), D191.2 (K), U23.3 (D2), U23.6 (D1)
- new net ROW6_INV3: D199.2 (K), D207.2 (K), D215.2 (K), D223.2 (K), D231.2 (K), D239.2 (K), D247.2 (K), D255.2 (K), U31.3 (D2), U31.6 (D1)
- new net ROW7_INV0: D16.2 (K), D24.2 (K), D32.2 (K), D40.2 (K), D48.2 (K), D56.2 (K), D64.2 (K), D8.2 (K), U8.3 (D2), U8.6 (D1)
- new net ROW7_INV1: D104.2 (K), D112.2 (K), D120.2 (K), D128.2 (K), D72.2 (K), D80.2 (K), D88.2 (K), D96.2 (K), U16.3 (D2), U16.6 (D1)
- new net ROW7_INV2: D136.2 (K), D144.2 (K), D152.2 (K), D160.2 (K), D168.2 (K), D176.2 (K), D184.2 (K), D192.2 (K), U24.3 (D2), U24.6 (D1)
- new net ROW7_INV3: D200.2 (K), D208.2 (K), D216.2 (K), D224.2 (K), D232.2 (K), D240.2 (K), D248.2 (K), D256.2 (K), U32.3 (D2), U32.6 (D1)
Other:
- note added: "INVERTING BUFFERS (lLED CATHODES)"
- moved on the sheet: C1, C2, C3, C4, P1, P2, P3, P4
