File: atmega328/four_panel/20mm_matrix/ver4/driver/driver.kicad_pcb (KiCad board)
At the start: 4 copper layers, 40 x 40 mm, 88 parts, among them IC1 ATMEGA328P-M, IC2 ATMEGA328P-M, IC3 ATMEGA328P-M, IC4 ATMEGA328P-M, P1 CONN_2X2, P2 CONN_2X2, P3 CONN_2X2, P4 CONN_2X2, U1 DMC2400UV, U10 DMC2400UV, U11 DMC2400UV, U12 DMC2400UV, U13 DMC2400UV, U14 DMC2400UV, U15 DMC2400UV, U16 DMC2400UV, U17 DMC2400UV, U18 DMC2400UV, U19 DMC2400UV, U2 DMC2400UV, U20 DMC2400UV, U21 DMC2400UV, U22 DMC2400UV, U23 DMC2400UV, U24 DMC2400UV, U25 DMC2400UV, U26 DMC2400UV, U27 DMC2400UV, U28 DMC2400UV, U29 DMC2400UV, U3 DMC2400UV, U30 DMC2400UV, U31 DMC2400UV, U32 DMC2400UV, U4 DMC2400UV, U5 DMC2400UV, U6 DMC2400UV, U7 DMC2400UV, U8 DMC2400UV, U9 DMC2400UV, X1 CER_RESO, X2 CER_RESO, X3 CER_RESO, X4 CER_RESO

Commit message: Worked on atmega328 4x20mm ver4. Modified silkscreen. Modified BOM changes 1% 82 Ohm resistor to 0.1% 160 Ohm resistor.
Parts:
- R10, R11, R12, R13, R14, R15, R16, R17, R18, R19, R20, R21, R22, R23, R24, R25, R26, R27, R28, R29, R30, R31, R32, R33, R34, R35, R36, R5, R6, R7, R8, R9: value 82 -> 160
Changed lines of the file:
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@@
     (links 337)
     (no_connects 0)
-    (area 49.392116 49.47125 90.212334 90.176601)
+    (area 48.376116 49.47125 90.212334 90.176601)
     (thickness 1.6)
     (drawings 15)
@@
       (effects (font (size 0.50038 0.4572) (thickness 0.1143)))
     )
-    (fp_text value 82 (at -1.69926 0 90) (layer F.SilkS) hide
+    (fp_text value 160 (at -1.69926 0 90) (layer F.SilkS) hide
       (effects (font (size 0.508 0.4572) (thickness 0.1143)))
     )
@@
       (effects (font (size 0.50038 0.4572) (thickness 0.1143)))
     )
-    (fp_text value 82 (at -1.69926 0 90) (layer F.SilkS) hide
+    (fp_text value 160 (at -1.69926 0 90) (layer F.SilkS) hide
       (effects (font (size 0.508 0.4572) (thickness 0.1143)))
     )
@@
       (effects (font (size 0.50038 0.4572) (thickness 0.1143)))
     )
-    (fp_text value 82 (at -1.69926 0 90) (layer F.SilkS) hide
+    (fp_text value 160 (at -1.69926 0 90) (layer F.SilkS) hide
       (effects (font (size 0.508 0.4572) (thickness 0.1143)))
     )
@@
       (effects (font (size 0.50038 0.4572) (thickness 0.1143)))
     )
-    (fp_text value 82 (at -1.69926 0 360) (layer F.SilkS) hide
+    (fp_text value 160 (at -1.69926 0 360) (layer F.SilkS) hide
       (effects (font (size 0.508 0.4572) (thickness 0.1143)))
     )
@@
       (effects (font (size 0.50038 0.4572) (thickness 0.1143)))
     )
-    (fp_text value 82 (at -1.69926 0 270) (layer F.SilkS) hide
+    (fp_text value 160 (at -1.69926 0 270) (layer F.SilkS) hide
       (effects (font (size 0.508 0.4572) (thickness 0.1143)))
     )
@@
       (effects (font (size 0.50038 0.4572) (thickness 0.1143)))
     )
-    (fp_text value 82 (at -1.69926 0 270) (layer F.SilkS) hide
+    (fp_text value 160 (at -1.69926 0 270) (layer F.SilkS) hide
       (effects (font (size 0.508 0.4572) (thickness 0.1143)))
     )
@@
       (effects (font (size 0.50038 0.4572) (thickness 0.1143)))
     )
-    (fp_text value 82 (at -1.69926 0 270) (layer F.SilkS) hide
+    (fp_text value 160 (at -1.69926 0 270) (layer F.SilkS) hide
       (effects (font (size 0.508 0.4572) (thickness 0.1143)))
     )
@@
       (effects (font (size 0.50038 0.4572) (thickness 0.1143)))
     )
-    (fp_text value 82 (at -1.69926 0 360) (layer F.SilkS) hide
+    (fp_text value 160 (at -1.69926 0 360) (layer F.SilkS) hide
       (effects (font (size 0.508 0.4572) (thickness 0.1143)))
     )
@@
       (effects (font (size 0.50038 0.4572) (thickness 0.1143)))
     )
-    (fp_text value 82 (at -1.69926 0 90) (layer F.SilkS) hide
+    (fp_text value 160 (at -1.69926 0 90) (layer F.SilkS) hide
       (effects (font (size 0.508 0.4572) (thickness 0.1143)))
     )
@@
       (effects (font (size 0.50038 0.4572) (thickness 0.1143)))
     )
-    (fp_text value 82 (at -1.69926 0 180) (layer F.SilkS) hide
+    (fp_text value 160 (at -1.69926 0 180) (layer F.SilkS) hide
       (effects (font (size 0.508 0.4572) (thickness 0.1143)))
     )
@@
       (effects (font (size 0.50038 0.4572) (thickness 0.1143)))
     )
-    (fp_text value 82 (at -1.69926 0 90) (layer F.SilkS) hide
+    (fp_text value 160 (at -1.69926 0 90) (layer F.SilkS) hide
       (effects (font (size 0.508 0.4572) (thickness 0.1143)))
     )
@@
       (effects (font (size 0.50038 0.4572) (thickness 0.1143)))
     )
-    (fp_text value 82 (at -1.69926 0 90) (layer F.SilkS) hide
+    (fp_text value 160 (at -1.69926 0 90) (layer F.SilkS) hide
       (effects (font (size 0.508 0.4572) (thickness 0.1143)))
     )
@@
       (effects (font (size 0.50038 0.4572) (thickness 0.1143)))
     )
-    (fp_text value 82 (at -1.69926 0 90) (layer F.SilkS) hide
+    (fp_text value 160 (at -1.69926 0 90) (layer F.SilkS) hide
       (effects (font (size 0.508 0.4572) (thickness 0.1143)))
     )
@@
       (effects (font (size 0.50038 0.4572) (thickness 0.1143)))
     )
-    (fp_text value 82 (at -1.69926 0 90) (layer F.SilkS) hide
+    (fp_text value 160 (at -1.69926 0 90) (layer F.SilkS) hide
       (effects (font (size 0.508 0.4572) (thickness 0.1143)))
     )
@@
       (effects (font (size 0.50038 0.4572) (thickness 0.1143)))
     )
-    (fp_text value 82 (at -1.69926 0 90) (layer F.SilkS) hide
+    (fp_text value 160 (at -1.69926 0 90) (layer F.SilkS) hide
       (effects (font (size 0.508 0.4572) (thickness 0.1143)))
     )
@@
       (effects (font (size 0.50038 0.4572) (thickness 0.1143)))
     )
-    (fp_text value 82 (at -1.69926 0 90) (layer F.SilkS) hide
+    (fp_text value 160 (at -1.69926 0 90) (layer F.SilkS) hide
       (effects (font (size 0.508 0.4572) (thickness 0.1143)))
     )
@@
       (effects (font (size 0.50038 0.4572) (thickness 0.1143)))
     )
-    (fp_text value 82 (at -1.69926 0 90) (layer F.SilkS) hide
+    (fp_text value 160 (at -1.69926 0 90) (layer F.SilkS) hide
       (effects (font (size 0.508 0.4572) (thickness 0.1143)))
     )
@@
       (effects (font (size 0.50038 0.4572) (thickness 0.1143)))
     )
-    (fp_text value 82 (at -1.69926 0 90) (layer F.SilkS) hide
+    (fp_text value 160 (at -1.69926 0 90) (layer F.SilkS) hide
       (effects (font (size 0.508 0.4572) (thickness 0.1143)))
     )
@@
       (effects (font (size 0.50038 0.4572) (thickness 0.1143)))
     )
-    (fp_text value 82 (at -1.69926 0 90) (layer F.SilkS) hide
+    (fp_text value 160 (at -1.69926 0 90) (layer F.SilkS) hide
       (effects (font (size 0.508 0.4572) (thickness 0.1143)))
     )
@@
       (effects (font (size 0.50038 0.4572) (thickness 0.1143)))
     )
-    (fp_text value 82 (at -1.69926 0 270) (layer F.SilkS) hide
+    (fp_text value 160 (at -1.69926 0 270) (layer F.SilkS) hide
       (effects (font (size 0.508 0.4572) (thickness 0.1143)))
     )
@@
       (effects (font (size 0.50038 0.4572) (thickness 0.1143)))
     )
-    (fp_text value 82 (at -1.69926 0 270) (layer F.SilkS) hide
+    (fp_text value 160 (at -1.69926 0 270) (layer F.SilkS) hide
       (effects (font (size 0.508 0.4572) (thickness 0.1143)))
     )
@@
       (effects (font (size 0.50038 0.4572) (thickness 0.1143)))
     )
-    (fp_text value 82 (at -1.69926 0 270) (layer F.SilkS) hide
+    (fp_text value 160 (at -1.69926 0 270) (layer F.SilkS) hide
       (effects (font (size 0.508 0.4572) (thickness 0.1143)))
     )
@@
       (effects (font (size 0.50038 0.4572) (thickness 0.1143)))
     )
-    (fp_text value 82 (at -1.69926 0 270) (layer F.SilkS) hide
+    (fp_text value 160 (at -1.69926 0 270) (layer F.SilkS) hide
       (effects (font (size 0.508 0.4572) (thickness 0.1143)))
     )
@@
       (effects (font (size 0.50038 0.4572) (thickness 0.1143)))
     )
-    (fp_text value 82 (at -1.69926 0 270) (layer F.SilkS) hide
+    (fp_text value 160 (at -1.69926 0 270) (layer F.SilkS) hide
       (effects (font (size 0.508 0.4572) (thickness 0.1143)))
     )
@@
       (effects (font (size 0.50038 0.4572) (thickness 0.1143)))
     )
-    (fp_text value 82 (at -1.69926 0 270) (layer F.SilkS) hide
+    (fp_text value 160 (at -1.69926 0 270) (layer F.SilkS) hide
       (effects (font (size 0.508 0.4572) (thickness 0.1143)))
     )
@@
       (effects (font (size 0.50038 0.4572) (thickness 0.1143)))
     )
-    (fp_text value 82 (at -1.69926 0 270) (layer F.SilkS) hide
+    (fp_text value 160 (at -1.69926 0 270) (layer F.SilkS) hide
       (effects (font (size 0.508 0.4572) (thickness 0.1143)))
     )
@@
       (effects (font (size 0.50038 0.4572) (thickness 0.1143)))
     )
-    (fp_text value 82 (at -1.69926 0 270) (layer F.SilkS) hide
+    (fp_text value 160 (at -1.69926 0 270) (layer F.SilkS) hide
       (effects (font (size 0.508 0.4572) (thickness 0.1143)))
     )
@@
       (effects (font (size 0.50038 0.4572) (thickness 0.1143)))
     )
-    (fp_text value 82 (at -1.69926 0 270) (layer F.SilkS) hide
+    (fp_text value 160 (at -1.69926 0 270) (layer F.SilkS) hide
       (effects (font (size 0.508 0.4572) (thickness 0.1143)))
     )
@@
       (effects (font (size 0.50038 0.4572) (thickness 0.1143)))
     )
-    (fp_text value 82 (at -1.69926 0 90) (layer F.SilkS) hide
+    (fp_text value 160 (at -1.69926 0 90) (layer F.SilkS) hide
       (effects (font (size 0.508 0.4572) (thickness 0.1143)))
     )
@@
       (effects (font (size 0.50038 0.4572) (thickness 0.1143)))
     )
-    (fp_text value 82 (at -1.69926 0 270) (layer F.SilkS) hide
+    (fp_text value 160 (at -1.69926 0 270) (layer F.SilkS) hide
       (effects (font (size 0.508 0.4572) (thickness 0.1143)))
     )
@@
       (effects (font (size 0.50038 0.4572) (thickness 0.1143)))
     )
-    (fp_text value 82 (at -1.69926 0 270) (layer F.SilkS) hide
+    (fp_text value 160 (at -1.69926 0 270) (layer F.SilkS) hide
       (effects (font (size 0.508 0.4572) (thickness 0.1143)))
     )
@@
       (effects (font (size 0.50038 0.4572) (thickness 0.1143)))
     )
-    (fp_text value 82 (at -1.69926 0 270) (layer F.SilkS) hide
-      (effects (font (size 0.508 0.4572) (thickness 0.1143)))
-    )
+    (fp_text value 160 (at -1.69926 0 270) (layer F.SilkS) hide
+      (effects (font (size 0.508 0.4572) (thickness 0.1143)))
+    )
