File: atmega328/four_panel/20mm_matrix/ver4/driver/driver.sch (KiCad schematic (older format))
At the start: 88 parts, among them IC1 ATMEGA328P-M, IC2 ATMEGA328P-M, IC3 ATMEGA328P-M, IC4 ATMEGA328P-M, P1 CONN_2X2, P2 CONN_2X2, P3 CONN_2X2, P4 CONN_2X2, U1 DMC2400UV, U10 DMC2400UV, U11 DMC2400UV, U12 DMC2400UV, U13 DMC2400UV, U14 DMC2400UV, U15 DMC2400UV, U16 DMC2400UV, U17 DMC2400UV, U18 DMC2400UV, U19 DMC2400UV, U2 DMC2400UV, U20 DMC2400UV, U21 DMC2400UV, U22 DMC2400UV, U23 DMC2400UV, U24 DMC2400UV, U25 DMC2400UV, U26 DMC2400UV, U27 DMC2400UV, U28 DMC2400UV, U29 DMC2400UV, U3 DMC2400UV, U30 DMC2400UV, U31 DMC2400UV, U32 DMC2400UV, U4 DMC2400UV, U5 DMC2400UV, U6 DMC2400UV, U7 DMC2400UV, U8 DMC2400UV, U9 DMC2400UV, X1 CER_RESO, X2 CER_RESO, X3 CER_RESO, X4 CER_RESO

Commit message: Added gerber files for new v0.4 version of driver design.
Parts:
- R10, R11, R12, R13, R14, R15, R16, R17, R18, R19, R20, R21, R22, R23, R24, R25, R26, R27, R28, R29, R30, R31, R32, R33, R34, R35, R36, R5, R6, R7, R8, R9: value 180 -> 82
Changed lines of the file:
@@
 Sheet 1 1
 Title ""
-Date "22 may 2016"
+Date "10 aug 2016"
 Rev ""
 Comp ""
@@
 P 2150 7200
 F 0 "R6" V 2230 7200 40  0000 C CNN
-F 1 "180" V 2157 7201 40  0000 C CNN
+F 1 "82" V 2157 7201 40  0000 C CNN
 F 2 "" V 2080 7200 30  0000 C CNN
 F 3 "" H 2150 7200 30  0000 C CNN
@@
 P 2350 7200
 F 0 "R7" V 2430 7200 40  0000 C CNN
-F 1 "180" V 2357 7201 40  0000 C CNN
+F 1 "82" V 2357 7201 40  0000 C CNN
 F 2 "" V 2280 7200 30  0000 C CNN
 F 3 "" H 2350 7200 30  0000 C CNN
@@
 P 1950 7200
 F 0 "R5" V 2030 7200 40  0000 C CNN
-F 1 "180" V 1957 7201 40  0000 C CNN
+F 1 "82" V 1957 7201 40  0000 C CNN
 F 2 "" V 1880 7200 30  0000 C CNN
 F 3 "" H 1950 7200 30  0000 C CNN
@@
 P 2550 7200
 F 0 "R8" V 2630 7200 40  0000 C CNN
-F 1 "180" V 2557 7201 40  0000 C CNN
+F 1 "82" V 2557 7201 40  0000 C CNN
 F 2 "" V 2480 7200 30  0000 C CNN
 F 3 "" H 2550 7200 30  0000 C CNN
@@
 P 2750 7200
 F 0 "R9" V 2830 7200 40  0000 C CNN
-F 1 "180" V 2757 7201 40  0000 C CNN
+F 1 "82" V 2757 7201 40  0000 C CNN
 F 2 "" V 2680 7200 30  0000 C CNN
 F 3 "" H 2750 7200 30  0000 C CNN
@@
 P 2950 7200
 F 0 "R10" V 3030 7200 40  0000 C CNN
-F 1 "180" V 2957 7201 40  0000 C CNN
+F 1 "82" V 2957 7201 40  0000 C CNN
 F 2 "" V 2880 7200 30  0000 C CNN
 F 3 "" H 2950 7200 30  0000 C CNN
@@
 P 3150 7200
 F 0 "R11" V 3230 7200 40  0000 C CNN
-F 1 "180" V 3157 7201 40  0000 C CNN
+F 1 "82" V 3157 7201 40  0000 C CNN
 F 2 "" V 3080 7200 30  0000 C CNN
 F 3 "" H 3150 7200 30  0000 C CNN
@@
 P 3350 7200
 F 0 "R12" V 3430 7200 40  0000 C CNN
-F 1 "180" V 3357 7201 40  0000 C CNN
+F 1 "82" V 3357 7201 40  0000 C CNN
 F 2 "" V 3280 7200 30  0000 C CNN
 F 3 "" H 3350 7200 30  0000 C CNN
@@
 P 6350 7200
 F 0 "R14" V 6430 7200 40  0000 C CNN
-F 1 "180" V 6357 7201 40  0000 C CNN
+F 1 "82" V 6357 7201 40  0000 C CNN
 F 2 "" V 6280 7200 30  0000 C CNN
 F 3 "" H 6350 7200 30  0000 C CNN
@@
 P 6550 7200
 F 0 "R15" V 6630 7200 40  0000 C CNN
-F 1 "180" V 6557 7201 40  0000 C CNN
+F 1 "82" V 6557 7201 40  0000 C CNN
 F 2 "" V 6480 7200 30  0000 C CNN
 F 3 "" H 6550 7200 30  0000 C CNN
@@
 P 6150 7200
 F 0 "R13" V 6230 7200 40  0000 C CNN
-F 1 "180" V 6157 7201 40  0000 C CNN
+F 1 "82" V 6157 7201 40  0000 C CNN
 F 2 "" V 6080 7200 30  0000 C CNN
 F 3 "" H 6150 7200 30  0000 C CNN
@@
 P 6750 7200
 F 0 "R16" V 6830 7200 40  0000 C CNN
-F 1 "180" V 6757 7201 40  0000 C CNN
+F 1 "82" V 6757 7201 40  0000 C CNN
 F 2 "" V 6680 7200 30  0000 C CNN
 F 3 "" H 6750 7200 30  0000 C CNN
@@
 P 6950 7200
 F 0 "R17" V 7030 7200 40  0000 C CNN
-F 1 "180" V 6957 7201 40  0000 C CNN
+F 1 "82" V 6957 7201 40  0000 C CNN
 F 2 "" V 6880 7200 30  0000 C CNN
 F 3 "" H 6950 7200 30  0000 C CNN
@@
 P 7150 7200
 F 0 "R18" V 7230 7200 40  0000 C CNN
-F 1 "180" V 7157 7201 40  0000 C CNN
+F 1 "82" V 7157 7201 40  0000 C CNN
 F 2 "" V 7080 7200 30  0000 C CNN
 F 3 "" H 7150 7200 30  0000 C CNN
@@
 P 7350 7200
 F 0 "R19" V 7430 7200 40  0000 C CNN
-F 1 "180" V 7357 7201 40  0000 C CNN
+F 1 "82" V 7357 7201 40  0000 C CNN
 F 2 "" V 7280 7200 30  0000 C CNN
 F 3 "" H 7350 7200 30  0000 C CNN
@@
 P 7550 7200
 F 0 "R20" V 7630 7200 40  0000 C CNN
-F 1 "180" V 7557 7201 40  0000 C CNN
+F 1 "82" V 7557 7201 40  0000 C CNN
 F 2 "" V 7480 7200 30  0000 C CNN
 F 3 "" H 7550 7200 30  0000 C CNN
@@
 P 10750 7200
 F 0 "R22" V 10830 7200 40  0000 C CNN
-F 1 "180" V 10757 7201 40  0000 C CNN
+F 1 "82" V 10757 7201 40  0000 C CNN
 F 2 "" V 10680 7200 30  0000 C CNN
 F 3 "" H 10750 7200 30  0000 C CNN
@@
 P 10950 7200
 F 0 "R23" V 11030 7200 40  0000 C CNN
-F 1 "180" V 10957 7201 40  0000 C CNN
+F 1 "82" V 10957 7201 40  0000 C CNN
 F 2 "" V 10880 7200 30  0000 C CNN
 F 3 "" H 10950 7200 30  0000 C CNN
@@
 P 10550 7200
 F 0 "R21" V 10630 7200 40  0000 C CNN
-F 1 "180" V 10557 7201 40  0000 C CNN
+F 1 "82" V 10557 7201 40  0000 C CNN
 F 2 "" V 10480 7200 30  0000 C CNN
 F 3 "" H 10550 7200 30  0000 C CNN
@@
 P 11150 7200
 F 0 "R24" V 11230 7200 40  0000 C CNN
-F 1 "180" V 11157 7201 40  0000 C CNN
+F 1 "82" V 11157 7201 40  0000 C CNN
 F 2 "" V 11080 7200 30  0000 C CNN
 F 3 "" H 11150 7200 30  0000 C CNN
@@
 P 11350 7200
 F 0 "R25" V 11430 7200 40  0000 C CNN
-F 1 "180" V 11357 7201 40  0000 C CNN
+F 1 "82" V 11357 7201 40  0000 C CNN
 F 2 "" V 11280 7200 30  0000 C CNN
 F 3 "" H 11350 7200 30  0000 C CNN
@@
 P 11550 7200
 F 0 "R26" V 11630 7200 40  0000 C CNN
-F 1 "180" V 11557 7201 40  0000 C CNN
+F 1 "82" V 11557 7201 40  0000 C CNN
 F 2 "" V 11480 7200 30  0000 C CNN
 F 3 "" H 11550 7200 30  0000 C CNN
@@
 P 11750 7200
 F 0 "R27" V 11830 7200 40  0000 C CNN
-F 1 "180" V 11757 7201 40  0000 C CNN
+F 1 "82" V 11757 7201 40  0000 C CNN
 F 2 "" V 11680 7200 30  0000 C CNN
 F 3 "" H 11750 7200 30  0000 C CNN
@@
 P 11950 7200
 F 0 "R28" V 12030 7200 40  0000 C CNN
-F 1 "180" V 11957 7201 40  0000 C CNN
+F 1 "82" V 11957 7201 40  0000 C CNN
 F 2 "" V 11880 7200 30  0000 C CNN
 F 3 "" H 11950 7200 30  0000 C CNN
@@
 P 14950 7200
 F 0 "R30" V 15030 7200 40  0000 C CNN
-F 1 "180" V 14957 7201 40  0000 C CNN
+F 1 "82" V 14957 7201 40  0000 C CNN
 F 2 "" V 14880 7200 30  0000 C CNN
 F 3 "" H 14950 7200 30  0000 C CNN
@@
 P 15150 7200
 F 0 "R31" V 15230 7200 40  0000 C CNN
-F 1 "180" V 15157 7201 40  0000 C CNN
+F 1 "82" V 15157 7201 40  0000 C CNN
 F 2 "" V 15080 7200 30  0000 C CNN
 F 3 "" H 15150 7200 30  0000 C CNN
@@
 P 14750 7200
 F 0 "R29" V 14830 7200 40  0000 C CNN
-F 1 "180" V 14757 7201 40  0000 C CNN
+F 1 "82" V 14757 7201 40  0000 C CNN
 F 2 "" V 14680 7200 30  0000 C CNN
 F 3 "" H 14750 7200 30  0000 C CNN
@@
 P 15350 7200
 F 0 "R32" V 15430 7200 40  0000 C CNN
-F 1 "180" V 15357 7201 40  0000 C CNN
+F 1 "82" V 15357 7201 40  0000 C CNN
 F 2 "" V 15280 7200 30  0000 C CNN
 F 3 "" H 15350 7200 30  0000 C CNN
@@
 P 15550 7200
 F 0 "R33" V 15630 7200 40  0000 C CNN
-F 1 "180" V 15557 7201 40  0000 C CNN
+F 1 "82" V 15557 7201 40  0000 C CNN
 F 2 "" V 15480 7200 30  0000 C CNN
 F 3 "" H 15550 7200 30  0000 C CNN
@@
 P 15750 7200
 F 0 "R34" V 15830 7200 40  0000 C CNN
-F 1 "180" V 15757 7201 40  0000 C CNN
+F 1 "82" V 15757 7201 40  0000 C CNN
 F 2 "" V 15680 7200 30  0000 C CNN
 F 3 "" H 15750 7200 30  0000 C CNN
@@
 P 15950 7200
 F 0 "R35" V 16030 7200 40  0000 C CNN
-F 1 "180" V 15957 7201 40  0000 C CNN
+F 1 "82" V 15957 7201 40  0000 C CNN
 F 2 "" V 15880 7200 30  0000 C CNN
 F 3 "" H 15950 7200 30  0000 C CNN
@@
 P 16150 7200
 F 0 "R36" V 16230 7200 40  0000 C CNN
-F 1 "180" V 16157 7201 40  0000 C CNN
+F 1 "82" V 16157 7201 40  0000 C CNN
 F 2 "" V 16080 7200 30  0000 C CNN
 F 3 "" H 16150 7200 30  0000 C CNN

Commit message: Worked on atmega328 4x20mm ver4. Modified silkscreen. Modified BOM changes 1% 82 Ohm resistor to 0.1% 160 Ohm resistor.
Parts:
- R10, R11, R12, R13, R14, R15, R16, R17, R18, R19, R20, R21, R22, R23, R24, R25, R26, R27, R28, R29, R30, R31, R32, R33, R34, R35, R36, R5, R6, R7, R8, R9: value 82 -> 160
Changed lines of the file:
@@
 Sheet 1 1
 Title ""
-Date "10 aug 2016"
+Date "5 dec 2016"
 Rev ""
 Comp ""
@@
 P 2150 7200
 F 0 "R6" V 2230 7200 40  0000 C CNN
-F 1 "82" V 2157 7201 40  0000 C CNN
+F 1 "160" V 2157 7201 40  0000 C CNN
 F 2 "" V 2080 7200 30  0000 C CNN
 F 3 "" H 2150 7200 30  0000 C CNN
@@
 P 2350 7200
 F 0 "R7" V 2430 7200 40  0000 C CNN
-F 1 "82" V 2357 7201 40  0000 C CNN
+F 1 "160" V 2357 7201 40  0000 C CNN
 F 2 "" V 2280 7200 30  0000 C CNN
 F 3 "" H 2350 7200 30  0000 C CNN
@@
 P 1950 7200
 F 0 "R5" V 2030 7200 40  0000 C CNN
-F 1 "82" V 1957 7201 40  0000 C CNN
+F 1 "160" V 1957 7201 40  0000 C CNN
 F 2 "" V 1880 7200 30  0000 C CNN
 F 3 "" H 1950 7200 30  0000 C CNN
@@
 P 2550 7200
 F 0 "R8" V 2630 7200 40  0000 C CNN
-F 1 "82" V 2557 7201 40  0000 C CNN
+F 1 "160" V 2557 7201 40  0000 C CNN
 F 2 "" V 2480 7200 30  0000 C CNN
 F 3 "" H 2550 7200 30  0000 C CNN
@@
 P 2750 7200
 F 0 "R9" V 2830 7200 40  0000 C CNN
-F 1 "82" V 2757 7201 40  0000 C CNN
+F 1 "160" V 2757 7201 40  0000 C CNN
 F 2 "" V 2680 7200 30  0000 C CNN
 F 3 "" H 2750 7200 30  0000 C CNN
@@
 P 2950 7200
 F 0 "R10" V 3030 7200 40  0000 C CNN
-F 1 "82" V 2957 7201 40  0000 C CNN
+F 1 "160" V 2957 7201 40  0000 C CNN
 F 2 "" V 2880 7200 30  0000 C CNN
 F 3 "" H 2950 7200 30  0000 C CNN
@@
 P 3150 7200
 F 0 "R11" V 3230 7200 40  0000 C CNN
-F 1 "82" V 3157 7201 40  0000 C CNN
+F 1 "160" V 3157 7201 40  0000 C CNN
 F 2 "" V 3080 7200 30  0000 C CNN
 F 3 "" H 3150 7200 30  0000 C CNN
@@
 P 3350 7200
 F 0 "R12" V 3430 7200 40  0000 C CNN
-F 1 "82" V 3357 7201 40  0000 C CNN
+F 1 "160" V 3357 7201 40  0000 C CNN
 F 2 "" V 3280 7200 30  0000 C CNN
 F 3 "" H 3350 7200 30  0000 C CNN
@@
 P 6350 7200
 F 0 "R14" V 6430 7200 40  0000 C CNN
-F 1 "82" V 6357 7201 40  0000 C CNN
+F 1 "160" V 6357 7201 40  0000 C CNN
 F 2 "" V 6280 7200 30  0000 C CNN
 F 3 "" H 6350 7200 30  0000 C CNN
@@
 P 6550 7200
 F 0 "R15" V 6630 7200 40  0000 C CNN
-F 1 "82" V 6557 7201 40  0000 C CNN
+F 1 "160" V 6557 7201 40  0000 C CNN
 F 2 "" V 6480 7200 30  0000 C CNN
 F 3 "" H 6550 7200 30  0000 C CNN
@@
 P 6150 7200
 F 0 "R13" V 6230 7200 40  0000 C CNN
-F 1 "82" V 6157 7201 40  0000 C CNN
+F 1 "160" V 6157 7201 40  0000 C CNN
 F 2 "" V 6080 7200 30  0000 C CNN
 F 3 "" H 6150 7200 30  0000 C CNN
@@
 P 6750 7200
 F 0 "R16" V 6830 7200 40  0000 C CNN
-F 1 "82" V 6757 7201 40  0000 C CNN
+F 1 "160" V 6757 7201 40  0000 C CNN
 F 2 "" V 6680 7200 30  0000 C CNN
 F 3 "" H 6750 7200 30  0000 C CNN
@@
 P 6950 7200
 F 0 "R17" V 7030 7200 40  0000 C CNN
-F 1 "82" V 6957 7201 40  0000 C CNN
+F 1 "160" V 6957 7201 40  0000 C CNN
 F 2 "" V 6880 7200 30  0000 C CNN
 F 3 "" H 6950 7200 30  0000 C CNN
@@
 P 7150 7200
 F 0 "R18" V 7230 7200 40  0000 C CNN
-F 1 "82" V 7157 7201 40  0000 C CNN
+F 1 "160" V 7157 7201 40  0000 C CNN
 F 2 "" V 7080 7200 30  0000 C CNN
 F 3 "" H 7150 7200 30  0000 C CNN
@@
 P 7350 7200
 F 0 "R19" V 7430 7200 40  0000 C CNN
-F 1 "82" V 7357 7201 40  0000 C CNN
+F 1 "160" V 7357 7201 40  0000 C CNN
 F 2 "" V 7280 7200 30  0000 C CNN
 F 3 "" H 7350 7200 30  0000 C CNN
@@
 P 7550 7200
 F 0 "R20" V 7630 7200 40  0000 C CNN
-F 1 "82" V 7557 7201 40  0000 C CNN
+F 1 "160" V 7557 7201 40  0000 C CNN
 F 2 "" V 7480 7200 30  0000 C CNN
 F 3 "" H 7550 7200 30  0000 C CNN
@@
 P 10750 7200
 F 0 "R22" V 10830 7200 40  0000 C CNN
-F 1 "82" V 10757 7201 40  0000 C CNN
+F 1 "160" V 10757 7201 40  0000 C CNN
 F 2 "" V 10680 7200 30  0000 C CNN
 F 3 "" H 10750 7200 30  0000 C CNN
@@
 P 10950 7200
 F 0 "R23" V 11030 7200 40  0000 C CNN
-F 1 "82" V 10957 7201 40  0000 C CNN
+F 1 "160" V 10957 7201 40  0000 C CNN
 F 2 "" V 10880 7200 30  0000 C CNN
 F 3 "" H 10950 7200 30  0000 C CNN
@@
 P 10550 7200
 F 0 "R21" V 10630 7200 40  0000 C CNN
-F 1 "82" V 10557 7201 40  0000 C CNN
+F 1 "160" V 10557 7201 40  0000 C CNN
 F 2 "" V 10480 7200 30  0000 C CNN
 F 3 "" H 10550 7200 30  0000 C CNN
@@
 P 11150 7200
 F 0 "R24" V 11230 7200 40  0000 C CNN
-F 1 "82" V 11157 7201 40  0000 C CNN
+F 1 "160" V 11157 7201 40  0000 C CNN
 F 2 "" V 11080 7200 30  0000 C CNN
 F 3 "" H 11150 7200 30  0000 C CNN
@@
 P 11350 7200
 F 0 "R25" V 11430 7200 40  0000 C CNN
-F 1 "82" V 11357 7201 40  0000 C CNN
+F 1 "160" V 11357 7201 40  0000 C CNN
 F 2 "" V 11280 7200 30  0000 C CNN
 F 3 "" H 11350 7200 30  0000 C CNN
@@
 P 11550 7200
 F 0 "R26" V 11630 7200 40  0000 C CNN
-F 1 "82" V 11557 7201 40  0000 C CNN
+F 1 "160" V 11557 7201 40  0000 C CNN
 F 2 "" V 11480 7200 30  0000 C CNN
 F 3 "" H 11550 7200 30  0000 C CNN
@@
 P 11750 7200
 F 0 "R27" V 11830 7200 40  0000 C CNN
-F 1 "82" V 11757 7201 40  0000 C CNN
+F 1 "160" V 11757 7201 40  0000 C CNN
 F 2 "" V 11680 7200 30  0000 C CNN
 F 3 "" H 11750 7200 30  0000 C CNN
@@
 P 11950 7200
 F 0 "R28" V 12030 7200 40  0000 C CNN
-F 1 "82" V 11957 7201 40  0000 C CNN
+F 1 "160" V 11957 7201 40  0000 C CNN
 F 2 "" V 11880 7200 30  0000 C CNN
 F 3 "" H 11950 7200 30  0000 C CNN
@@
 P 14950 7200
 F 0 "R30" V 15030 7200 40  0000 C CNN
-F 1 "82" V 14957 7201 40  0000 C CNN
+F 1 "160" V 14957 7201 40  0000 C CNN
 F 2 "" V 14880 7200 30  0000 C CNN
 F 3 "" H 14950 7200 30  0000 C CNN
@@
 P 15150 7200
 F 0 "R31" V 15230 7200 40  0000 C CNN
-F 1 "82" V 15157 7201 40  0000 C CNN
+F 1 "160" V 15157 7201 40  0000 C CNN
 F 2 "" V 15080 7200 30  0000 C CNN
 F 3 "" H 15150 7200 30  0000 C CNN
@@
 P 14750 7200
 F 0 "R29" V 14830 7200 40  0000 C CNN
-F 1 "82" V 14757 7201 40  0000 C CNN
+F 1 "160" V 14757 7201 40  0000 C CNN
 F 2 "" V 14680 7200 30  0000 C CNN
 F 3 "" H 14750 7200 30  0000 C CNN
@@
 P 15350 7200
 F 0 "R32" V 15430 7200 40  0000 C CNN
-F 1 "82" V 15357 7201 40  0000 C CNN
+F 1 "160" V 15357 7201 40  0000 C CNN
 F 2 "" V 15280 7200 30  0000 C CNN
 F 3 "" H 15350 7200 30  0000 C CNN
@@
 P 15550 7200
 F 0 "R33" V 15630 7200 40  0000 C CNN
-F 1 "82" V 15557 7201 40  0000 C CNN
+F 1 "160" V 15557 7201 40  0000 C CNN
 F 2 "" V 15480 7200 30  0000 C CNN
 F 3 "" H 15550 7200 30  0000 C CNN
@@
 P 15750 7200
 F 0 "R34" V 15830 7200 40  0000 C CNN
-F 1 "82" V 15757 7201 40  0000 C CNN
+F 1 "160" V 15757 7201 40  0000 C CNN
 F 2 "" V 15680 7200 30  0000 C CNN
 F 3 "" H 15750 7200 30  0000 C CNN
@@
 P 15950 7200
 F 0 "R35" V 16030 7200 40  0000 C CNN
-F 1 "82" V 15957 7201 40  0000 C CNN
+F 1 "160" V 15957 7201 40  0000 C CNN
 F 2 "" V 15880 7200 30  0000 C CNN
 F 3 "" H 15950 7200 30  0000 C CNN
@@
 P 16150 7200
 F 0 "R36" V 16230 7200 40  0000 C CNN
-F 1 "82" V 16157 7201 40  0000 C CNN
+F 1 "160" V 16157 7201 40  0000 C CNN
 F 2 "" V 16080 7200 30  0000 C CNN
 F 3 "" H 16150 7200 30  0000 C CNN
