File: helper/placeholder/placeholder.kicad_pcb (KiCad board)
At the start: 2 copper layers, 40 x 40 mm, 2 parts, among them J1 Conn_01x15_Male, J2 Conn_01x15_Female

Commit message: export v0.2, ready for production
Routing:
- net /EXT_INTO: track 26.7 -> 82.0 mm
- net /CS7: track 32.2 -> 82.0 mm
- net /CS6: track 37.3 -> 82.0 mm
- net /RESET: track 42.2 -> 82.0 mm
- net /CS5: track 46.5 -> 83.6 mm
- net /SCK: track 47.3 -> 81.9 mm
- net /CS4: track 54.3 -> 82.0 mm
- net /COPI: track 54.7 -> 82.0 mm
- net /CIPO: track 59.8 -> 82.0 mm
- net /CS3: track 60.0 -> 82.0 mm
- net /CS2: track 66.4 -> 82.0 mm
- net /CS1: track 72.1 -> 82.2 mm
Other:
- board text added: "G4 placeholder v0.2"
- board text removed: "G4 placeholder v0.1"
