File: atmega328/four_panel/20mm_matrix/ver3/programmer/prog_shield/prog_shield.sch (KiCad schematic (older format))
At the start: 3 parts, among them P1 CONN_3X2

Commit message: move driver to panel repo
Parts:
- C1: symbol CP1 -> prog_shield-rescue:CP1
- P1: symbol CONN_3X2 -> prog_shield-rescue:CONN_3X2
- SHIELD1: symbol ARDUINO_SHIELD -> arduino:ARDUINO_SHIELD
Connections:
- net RST: now also SHIELD1.10; no longer SHIELD1.RST
Changed lines of the file:
@@
-EESchema Schematic File Version 2
-LIBS:power
-LIBS:device
-LIBS:transistors
-LIBS:conn
-LIBS:linear
-LIBS:regul
-LIBS:74xx
-LIBS:cmos4000
-LIBS:adc-dac
-LIBS:memory
-LIBS:xilinx
-LIBS:special
-LIBS:microcontrollers
-LIBS:dsp
-LIBS:microchip
-LIBS:analog_switches
-LIBS:motorola
-LIBS:texas
-LIBS:intel
-LIBS:audio
-LIBS:interface
-LIBS:digital-audio
-LIBS:philips
-LIBS:display
-LIBS:cypress
-LIBS:siliconi
-LIBS:opto
-LIBS:atmel
-LIBS:contrib
-LIBS:valves
-LIBS:arduino
-LIBS:prog_shield-cache
-EELAYER 27 0
+EESchema Schematic File Version 4
+EELAYER 30 0
 EELAYER END
 $Descr A4 11693 8268
@@
 $EndDescr
 $Comp
-L ARDUINO_SHIELD SHIELD1
+L arduino:ARDUINO_SHIELD SHIELD1
 U 1 1 55D3A8F9
 P 3700 2600
@@
 $EndComp
 $Comp
-L CONN_3X2 P1
+L prog_shield-rescue:CONN_3X2 P1
 U 1 1 55D3A909
 P 6550 2500
@@
 $EndComp
 $Comp
-L CP1 C1
+L prog_shield-rescue:CP1 C1
 U 1 1 55D3A922
 P 1650 2400
@@
 	2750 2400 2500 2400
 Wire Wire Line
-	2750 2200 2500 2200
-Wire Wire Line
-	2500 2600 2750 2600
+	2500 2600 2650 2600
 Wire Wire Line
 	2650 2500 2750 2500
@@
 Wire Wire Line
 	4650 2200 4900 2200
-Text Label 2500 2200 2    60   ~ 0
+Text Label 4900 2300 0    60   ~ 0
 RST
 Text Label 2500 2400 2    60   ~ 0
@@
 NoConn ~ 4650 1800
 NoConn ~ 4650 1900
-NoConn ~ 4650 2300
+NoConn ~ 2750 2200
 NoConn ~ 4650 2400
 NoConn ~ 4650 2500
@@
 NoConn ~ 4650 3200
 $Comp
-L PWR_FLAG #FLG01
+L power:PWR_FLAG #FLG01
 U 1 1 55D3AC23
 P 8650 2450
@@
 $EndComp
 $Comp
-L PWR_FLAG #FLG02
+L power:PWR_FLAG #FLG02
 U 1 1 55D3AC32
 P 9200 2450
@@
 Text Label 9200 2600 3    60   ~ 0
 GND
+Wire Wire Line
+	2650 2600 2750 2600
+Wire Wire Line
+	4650 2300 4900 2300
 $EndSCHEMATC
