File: comm_placeholder_v0/comm_placeholder_v0.kicad_pcb (KiCad board)
At the start: 2 copper layers, 40 x 40 mm, 2 parts, among them J1 Conn_01x15_Male, J2 Conn_01x15_Female

Commit message: move placeholder
Parts:
- J1: footprint placeholdere-feet:HEADER_BOT -> comm_placeholder_v0:HEADER_BOT
- J2: footprint placeholdere-feet:HEADER_TOP -> comm_placeholder_v0:HEADER_TOP
