File: comm_v0p5/comm_v0p5.kicad_sch (KiCad schematic)
At the start: 14 parts, among them J1 1x15 header, J2 1x15 socket, J4 2x2 socket, J5 2x2 socket, J6 2x2 socket, J7 2x2 socket, U1 ATmega328PB-M, U2 AZ1117-5.0, Y1 20MHz

Commit message: Renamed comm_v0p4_opt2 to comm_v0p5.  Added JLCPCB BOM (minus global parts LCSC#s).
Parts:
- U2: DigiKey PN (none) -> AZ1117IH-5.0TRG1DITR-ND; PN (none) -> AZ1117IH-5.0TRG1
Changed lines of the file:
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@@
     (pin "2")
     (instances
-      (project "comm_v0p4"
+      (project "comm_v0p5"
         (path "/4a438c85-e5df-473f-b41d-177df9356b07"
           (reference "R5") (unit 1)
@@
     (pin "2")
     (instances
-      (project "comm_v0p4"
+      (project "comm_v0p5"
         (path "/4a438c85-e5df-473f-b41d-177df9356b07"
           (reference "C1") (unit 1)
@@
     (pin "1")
     (instances
-      (project "comm_v0p4"
+      (project "comm_v0p5"
         (path "/4a438c85-e5df-473f-b41d-177df9356b07"
           (reference "#PWR015") (unit 1)
@@
     (pin "4")
     (instances
-      (project "comm_v0p4"
+      (project "comm_v0p5"
         (path "/4a438c85-e5df-473f-b41d-177df9356b07"
           (reference "J5") (unit 1)
@@
     (pin "1")
     (instances
-      (project "comm_v0p4"
+      (project "comm_v0p5"
         (path "/4a438c85-e5df-473f-b41d-177df9356b07"
           (reference "#PWR014") (unit 1)
@@
     (pin "1")
     (instances
-      (project "comm_v0p4"
+      (project "comm_v0p5"
         (path "/4a438c85-e5df-473f-b41d-177df9356b07"
           (reference "#PWR011") (unit 1)
@@
     (pin "9")
     (instances
-      (project "comm_v0p4"
+      (project "comm_v0p5"
         (path "/4a438c85-e5df-473f-b41d-177df9356b07"
           (reference "J1") (unit 1)
@@
     (pin "1")
     (instances
-      (project "comm_v0p4"
+      (project "comm_v0p5"
         (path "/4a438c85-e5df-473f-b41d-177df9356b07"
           (reference "#PWR018") (unit 1)
@@
     (pin "9")
     (instances
-      (project "comm_v0p4"
+      (project "comm_v0p5"
         (path "/4a438c85-e5df-473f-b41d-177df9356b07"
           (reference "U1") (unit 1)
@@
     (pin "1")
     (instances
-      (project "comm_v0p4"
+      (project "comm_v0p5"
         (path "/4a438c85-e5df-473f-b41d-177df9356b07"
           (reference "#PWR09") (unit 1)
@@
     (pin "4")
     (instances
-      (project "comm_v0p4"
+      (project "comm_v0p5"
         (path "/4a438c85-e5df-473f-b41d-177df9356b07"
           (reference "J4") (unit 1)
@@
     (pin "1")
     (instances
-      (project "comm_v0p4"
+      (project "comm_v0p5"
         (path "/4a438c85-e5df-473f-b41d-177df9356b07"
           (reference "#PWR04") (unit 1)
@@
     (pin "1")
     (instances
-      (project "comm_v0p4"
+      (project "comm_v0p5"
         (path "/4a438c85-e5df-473f-b41d-177df9356b07"
           (reference "#PWR08") (unit 1)
@@
       (effects (font (size 1.27 1.27)) hide)
     )
+    (property "DigiKey PN" "AZ1117IH-5.0TRG1DITR-ND " (at 317.5 109.22 0)
+      (effects (font (size 1.27 1.27)) hide)
+    )
+    (property "PN" "AZ1117IH-5.0TRG1" (at 317.5 109.22 0)
+      (effects (font (size 1.27 1.27)) hide)
+    )
     (pin "1")
     (pin "2")
     (pin "3")
     (instances
-      (project "comm_v0p4"
+      (project "comm_v0p5"
         (path "/4a438c85-e5df-473f-b41d-177df9356b07"
           (reference "U2") (unit 1)
@@
     (pin "1")
     (instances
-      (project "comm_v0p4"
+      (project "comm_v0p5"
         (path "/4a438c85-e5df-473f-b41d-177df9356b07"
           (reference "#PWR03") (unit 1)
@@
     (pin "1")
     (instances
-      (project "comm_v0p4"
+      (project "comm_v0p5"
         (path "/4a438c85-e5df-473f-b41d-177df9356b07"
           (reference "#PWR016") (unit 1)
@@
     (pin "1")
     (instances
-      (project "comm_v0p4"
+      (project "comm_v0p5"
         (path "/4a438c85-e5df-473f-b41d-177df9356b07"
           (reference "#PWR013") (unit 1)
@@
     (pin "1")
     (instances
-      (project "comm_v0p4"
+      (project "comm_v0p5"
         (path "/4a438c85-e5df-473f-b41d-177df9356b07"
           (reference "#PWR02") (unit 1)
@@
     (pin "1")
     (instances
-      (project "comm_v0p4"
+      (project "comm_v0p5"
         (path "/4a438c85-e5df-473f-b41d-177df9356b07"
           (reference "#PWR07") (unit 1)
@@
     (pin "2")
     (instances
-      (project "comm_v0p4"
+      (project "comm_v0p5"
         (path "/4a438c85-e5df-473f-b41d-177df9356b07"
           (reference "C3") (unit 1)
@@
     (pin "2")
     (instances
-      (project "comm_v0p4"
+      (project "comm_v0p5"
         (path "/4a438c85-e5df-473f-b41d-177df9356b07"
           (reference "C4") (unit 1)
@@
     (pin "2")
     (instances
-      (project "comm_v0p4"
+      (project "comm_v0p5"
         (path "/4a438c85-e5df-473f-b41d-177df9356b07"
           (reference "C2") (unit 1)
@@
     (pin "4")
     (instances
-      (project "comm_v0p4"
+      (project "comm_v0p5"
         (path "/4a438c85-e5df-473f-b41d-177df9356b07"
           (reference "J6") (unit 1)
@@
     (pin "1")
     (instances
-      (project "comm_v0p4"
+      (project "comm_v0p5"
         (path "/4a438c85-e5df-473f-b41d-177df9356b07"
           (reference "#PWR019") (unit 1)
@@
     (pin "4")
     (instances
-      (project "comm_v0p4"
+      (project "comm_v0p5"
         (path "/4a438c85-e5df-473f-b41d-177df9356b07"
           (reference "J7") (unit 1)
@@
     (pin "1")
     (instances
-      (project "comm_v0p4"
+      (project "comm_v0p5"
         (path "/4a438c85-e5df-473f-b41d-177df9356b07"
           (reference "#PWR017") (unit 1)
@@
     (pin "1")
     (instances
-      (project "comm_v0p4"
+      (project "comm_v0p5"
         (path "/4a438c85-e5df-473f-b41d-177df9356b07"
           (reference "#PWR010") (unit 1)
@@
     (pin "1")
     (instances
-      (project "comm_v0p4"
+      (project "comm_v0p5"
         (path "/4a438c85-e5df-473f-b41d-177df9356b07"
           (reference "#FLG03") (unit 1)
@@
     (pin "1")
     (instances
-      (project "comm_v0p4"
+      (project "comm_v0p5"
         (path "/4a438c85-e5df-473f-b41d-177df9356b07"
           (reference "#PWR012") (unit 1)
@@
     (pin "1")
     (instances
-      (project "comm_v0p4"
+      (project "comm_v0p5"
         (path "/4a438c85-e5df-473f-b41d-177df9356b07"
           (reference "#FLG01") (unit 1)
@@
     (pin "1")
     (instances
-      (project "comm_v0p4"
+      (project "comm_v0p5"
         (path "/4a438c85-e5df-473f-b41d-177df9356b07"
           (reference "#PWR05") (unit 1)
@@
     (pin "9")
     (instances
-      (project "comm_v0p4"
+      (project "comm_v0p5"
         (path "/4a438c85-e5df-473f-b41d-177df9356b07"
           (reference "J2") (unit 1)
@@
     (pin "3")
     (instances
-      (project "comm_v0p4"
+      (project "comm_v0p5"
         (path "/4a438c85-e5df-473f-b41d-177df9356b07"
           (reference "Y1") (unit 1)
