File: comm_v0p6/comm_v0p6.kicad_pcb (KiCad board)
At the start: 4 copper layers, 40 x 40 mm, 12 parts, among them J1 1x15 header, J2 1x15 socket, J4 2x2 socket, J5 2x2 socket, J6 2x2 socket, J7 2x2 socket, U1 ATmega328PB-M, Y1 20MHz

Commit message: Completed projuction files for comm_v0p5
Routing:
- net /RESET_MSTR: track 57.1 -> 61.3 mm
- net /B0_SCK: track 54.2 -> 57.0 mm
- net /RESET_DRV2: track 13.9 -> 15.7 mm
- net /RESET_DRV3: track 31.3 -> 31.9 mm
Changed lines of the file:
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@@
   (segment (start 83.4779 60.628) (end 83.4779 81.8378) (width 0.2) (layer "B.Cu") (net 9))
   (segment (start 83.4779 81.8378) (end 85.24 83.5999) (width 0.2) (layer "B.Cu") (net 9))
-  (segment (start 64.92 83.7716) (end 65.151 83.5406) (width 0.2) (layer "F.Cu") (net 10))
+  (segment (start 64.92 83.543) (end 70.2358 78.2272) (width 0.2) (layer "F.Cu") (net 10))
   (segment (start 70.2358 78.2272) (end 70.2358 74.7331) (width 0.2) (layer "F.Cu") (net 10))
-  (segment (start 64.92 84.7) (end 64.92 83.7716) (width 0.2) (layer "F.Cu") (net 10))
-  (segment (start 65.151 83.312) (end 70.2358 78.2272) (width 0.2) (layer "F.Cu") (net 10))
-  (segment (start 65.151 83.5406) (end 65.151 83.312) (width 0.2) (layer "F.Cu") (net 10))
+  (segment (start 64.92 84.7) (end 64.92 83.543) (width 0.2) (layer "F.Cu") (net 10))
   (segment (start 65.151 84.469) (end 64.92 84.7) (width 0.2) (layer "F.Cu") (net 10))
   (segment (start 74.1426 77.3938) (end 64.6684 77.3938) (width 0.2) (layer "B.Cu") (net 10))
@@
   (segment (start 66.19 83.797) (end 71.208 78.779) (width 0.2) (layer "F.Cu") (net 12))
   (segment (start 71.208 78.779) (end 71.208 74.7331) (width 0.2) (layer "F.Cu") (net 12))
-  (segment (start 56.4618 65.636) (end 56.4618 61.9822) (width 0.2) (layer "B.Cu") (net 12))
+  (segment (start 57.6326 60.5028) (end 59.5376 60.5028) (width 0.2) (layer "B.Cu") (net 12))
+  (segment (start 59.84 84.7) (end 59.84 83.1064) (width 0.2) (layer "B.Cu") (net 12))
+  (segment (start 59.5376 60.5028) (end 59.84 60.2004) (width 0.2) (layer "B.Cu") (net 12))
+  (segment (start 52.2986 80.2894) (end 52.2986 69.7992) (width 0.2) (layer "B.Cu") (net 12))
+  (segment (start 54.1782 82.169) (end 52.2986 80.2894) (width 0.2) (layer "B.Cu") (net 12))
+  (segment (start 56.4618 61.6736) (end 57.6326 60.5028) (width 0.2) (layer "B.Cu") (net 12))
+  (segment (start 56.4618 65.636) (end 56.4618 61.6736) (width 0.2) (layer "B.Cu") (net 12))
+  (segment (start 59.84 60.2004) (end 59.84 58.75) (width 0.2) (layer "B.Cu") (net 12))
+  (segment (start 58.9026 82.169) (end 54.1782 82.169) (width 0.2) (layer "B.Cu") (net 12))
+  (segment (start 59.84 83.1064) (end 58.9026 82.169) (width 0.2) (layer "B.Cu") (net 12))
   (segment (start 52.2986 69.7992) (end 56.4618 65.636) (width 0.2) (layer "B.Cu") (net 12))
-  (segment (start 56.3761 80.9611) (end 56.3761 77.0517) (width 0.2) (layer "B.Cu") (net 12))
-  (segment (start 59.84 83.5999) (end 59.0149 83.5999) (width 0.2) (layer "B.Cu") (net 12))
-  (segment (start 58.7399 58.75) (end 59.84 58.75) (width 0.2) (layer "B.Cu") (net 12))
-  (segment (start 59.0149 83.5999) (end 56.3761 80.9611) (width 0.2) (layer "B.Cu") (net 12))
-  (segment (start 56.3761 77.0517) (end 52.2986 72.9742) (width 0.2) (layer "B.Cu") (net 12))
-  (segment (start 59.84 84.7) (end 59.84 83.5999) (width 0.2) (layer "B.Cu") (net 12))
-  (segment (start 58.7399 59.7041) (end 58.7399 58.75) (width 0.2) (layer "B.Cu") (net 12))
-  (segment (start 56.4618 61.9822) (end 58.7399 59.7041) (width 0.2) (layer "B.Cu") (net 12))
-  (segment (start 52.2986 72.9742) (end 52.2986 69.7992) (width 0.2) (layer "B.Cu") (net 12))
   (segment (start 58.8701 62.23) (end 70.5335 62.23) (width 0.2) (layer "F.Cu") (net 13))
   (segment (start 70.5335 62.23) (end 71.1918 62.8883) (width 0.2) (layer "F.Cu") (net 13))
@@
   (segment (start 70.0786 78.486) (end 71.0946 79.502) (width 0.2) (layer "B.Cu") (net 16))
   (segment (start 71.0946 79.502) (end 73.1266 79.502) (width 0.2) (layer "B.Cu") (net 16))
-  (segment (start 64.0551 70.1312) (end 56.3301 77.8562) (width 0.2) (layer "F.Cu") (net 17))
+  (segment (start 62.2282 70.1312) (end 55.23 77.1294) (width 0.2) (layer "F.Cu") (net 17))
+  (segment (start 64.0551 70.1312) (end 62.2282 70.1312) (width 0.2) (layer "F.Cu") (net 17))
   (segment (start 71.9151 69.5182) (end 72.4466 68.9867) (width 0.2) (layer "F.Cu") (net 17))
-  (segment (start 55.23 78.23) (end 56.3301 78.23) (width 0.2) (layer "F.Cu") (net 17))
   (segment (start 72.4466 68.9867) (end 72.4466 68.7795) (width 0.2) (layer "F.Cu") (net 17))
-  (segment (start 56.3301 77.8562) (end 56.3301 78.23) (width 0.2) (layer "F.Cu") (net 17))
+  (segment (start 55.23 77.1294) (end 55.23 78.23) (width 0.2) (layer "F.Cu") (net 17))
   (via (at 72.4466 68.7795) (size 0.6) (drill 0.3) (layers "F.Cu" "B.Cu") (net 17))
   (via (at 64.0551 70.1312) (size 0.6) (drill 0.3) (layers "F.Cu" "B.Cu") (net 17))
@@
   (segment (start 73.6829 72.2582) (end 74.213718 72.2582) (width 0.2) (layer "F.Cu") (net 22))
   (segment (start 75.3369 73.381382) (end 75.3369 76.0979) (width 0.2) (layer "F.Cu") (net 22))
-  (segment (start 84.77 64.77) (end 83.6699 64.77) (width 0.2) (layer "F.Cu") (net 23))
-  (segment (start 77.3818 71.286) (end 83.6699 64.9979) (width 0.2) (layer "F.Cu") (net 23))
-  (segment (start 73.6829 71.286) (end 77.3818 71.286) (width 0.2) (layer "F.Cu") (net 23))
-  (segment (start 83.6699 64.9979) (end 83.6699 64.77) (width 0.2) (layer "F.Cu") (net 23))
-  (segment (start 82.23 76.0882) (end 85.8943 72.4239) (width 0.2) (layer "F.Cu") (net 24))
-  (segment (start 85.8943 64.3042) (end 85.2346 63.6445) (width 0.2) (layer "F.Cu") (net 24))
-  (segment (start 85.2346 63.6445) (end 80.6173 63.6445) (width 0.2) (layer "F.Cu") (net 24))
+  (segment (start 84.77 64.77) (end 84.77 67.9602) (width 0.2) (layer "F.Cu") (net 23))
+  (segment (start 81.4442 71.286) (end 73.6829 71.286) (width 0.2) (layer "F.Cu") (net 23))
+  (segment (start 84.77 67.9602) (end 81.4442 71.286) (width 0.2) (layer "F.Cu") (net 23))
+  (segment (start 85.1916 63.4238) (end 80.838 63.4238) (width 0.2) (layer "F.Cu") (net 24))
+  (segment (start 86.3092 64.5414) (end 85.1916 63.4238) (width 0.2) (layer "F.Cu") (net 24))
+  (segment (start 80.838 63.4238) (end 73.3294 70.9324) (width 0.2) (layer "F.Cu") (net 24))
+  (segment (start 86.3092 72.009) (end 86.3092 64.5414) (width 0.2) (layer "F.Cu") (net 24))
+  (segment (start 82.23 76.0882) (end 86.3092 72.009) (width 0.2) (layer "F.Cu") (net 24))
   (segment (start 82.23 78.23) (end 82.23 76.0882) (width 0.2) (layer "F.Cu") (net 24))
-  (segment (start 80.6173 63.6445) (end 73.3294 70.9324) (width 0.2) (layer "F.Cu") (net 24))
-  (segment (start 85.8943 72.4239) (end 85.8943 64.3042) (width 0.2) (layer "F.Cu") (net 24))
-  (segment (start 58.4001 58.8876) (end 59.3626 59.8501) (width 0.2) (layer "F.Cu") (net 25))
+  (segment (start 57.3 58.75) (end 57.3 59.8654) (width 0.2) (layer "F.Cu") (net 25))
   (segment (start 72.0624 63.4466) (end 72.1614 63.3476) (width 0.2) (layer "F.Cu") (net 25))
-  (segment (start 59.3626 59.8501) (end 68.6639 59.8501) (width 0.2) (layer "F.Cu") (net 25))
-  (segment (start 68.6639 59.8501) (end 72.1614 63.3476) (width 0.2) (layer "F.Cu") (net 25))
-  (segment (start 58.4001 58.75) (end 58.4001 58.8876) (width 0.2) (layer "F.Cu") (net 25))
+  (segment (start 57.785 60.3504) (end 69.1642 60.3504) (width 0.2) (layer "F.Cu") (net 25))
+  (segment (start 69.1642 60.3504) (end 72.1614 63.3476) (width 0.2) (layer "F.Cu") (net 25))
   (segment (start 74.2971 67.8434) (end 72.2687 69.8718) (width 0.2) (layer "F.Cu") (net 25))
   (segment (start 72.0624 65.5574) (end 72.0624 63.4466) (width 0.2) (layer "F.Cu") (net 25))
-  (segment (start 57.3 58.75) (end 58.4001 58.75) (width 0.2) (layer "F.Cu") (net 25))
+  (segment (start 57.3 59.8654) (end 57.785 60.3504) (width 0.2) (layer "F.Cu") (net 25))
   (segment (start 74.3458 67.8434) (end 74.2971 67.8434) (width 0.2) (layer "F.Cu") (net 25))
   (via (at 72.0624 65.5574) (size 0.6) (drill 0.3) (layers "F.Cu" "B.Cu") (net 25))
   (via (at 74.3458 67.8434) (size 0.6) (drill 0.3) (layers "F.Cu" "B.Cu") (net 25))
-  (segment (start 51.5112 78.6696) (end 56.4415 83.5999) (width 0.2) (layer "B.Cu") (net 25))
+  (segment (start 52.7558 60.2996) (end 56.8452 60.2996) (width 0.2) (layer "B.Cu") (net 25))
+  (segment (start 56.8452 60.2996) (end 57.3 59.8448) (width 0.2) (layer "B.Cu") (net 25))
   (segment (start 74.3458 67.8434) (end 74.3458 67.8408) (width 0.2) (layer "B.Cu") (net 25))
-  (segment (start 56.1999 58.75) (end 56.1999 59.1806) (width 0.2) (layer "B.Cu") (net 25))
-  (segment (start 56.1999 59.1806) (end 51.5112 63.8693) (width 0.2) (layer "B.Cu") (net 25))
-  (segment (start 51.5112 63.8693) (end 51.5112 78.6696) (width 0.2) (layer "B.Cu") (net 25))
+  (segment (start 51.5112 81.8134) (end 51.5112 61.5442) (width 0.2) (layer "B.Cu") (net 25))
+  (segment (start 57.3 83.589) (end 57.0992 83.3882) (width 0.2) (layer "B.Cu") (net 25))
+  (segment (start 51.5112 61.5442) (end 52.7558 60.2996) (width 0.2) (layer "B.Cu") (net 25))
+  (segment (start 57.0992 83.3882) (end 53.086 83.3882) (width 0.2) (layer "B.Cu") (net 25))
+  (segment (start 57.3 84.7) (end 57.3 83.589) (width 0.2) (layer "B.Cu") (net 25))
   (segment (start 74.3458 67.8408) (end 72.0624 65.5574) (width 0.2) (layer "B.Cu") (net 25))
-  (segment (start 56.4415 83.5999) (end 57.3 83.5999) (width 0.2) (layer "B.Cu") (net 25))
-  (segment (start 57.3 58.75) (end 56.1999 58.75) (width 0.2) (layer "B.Cu") (net 25))
-  (segment (start 57.3 83.5999) (end 57.3 84.7) (width 0.2) (layer "B.Cu") (net 25))
+  (segment (start 57.3 59.8448) (end 57.3 58.75) (width 0.2) (layer "B.Cu") (net 25))
+  (segment (start 53.086 83.3882) (end 51.5112 81.8134) (width 0.2) (layer "B.Cu") (net 25))
   (segment (start 68.1144 70.9324) (end 66.7004 69.5184) (width 0.2) (layer "F.Cu") (net 26))
   (segment (start 66.7004 69.5184) (end 66.7004 69.459418) (width 0.2) (layer "F.Cu") (net 26))
